File: LattePanda_Module.kicad_sch (KiCad schematic)
At the start: 0 parts

Commit message: feat: Added hierarchical sheets and pins
Parts:
- added A1: LattePanda_Mu, Module_LattePanda:LattePanda_Module_H8.0mm_Horizontal, symbol MCU_Module_LattePanda:LattePanda_Mu
- added BT1: Battery_Cell, symbol Device:Battery_Cell
- added J1: Conn_01x03_Pin, A_HDJ_Library:PinHeader_1x03_P2.54mm_Vertical, symbol Connector:Conn_01x03_Pin
- added R1: 1k/1%, symbol Device:R
- added R2, R78, R79: 10k/1%, symbol Device:R
- added R76, R77: 100k/1%, symbol Device:R
- added TP78: TestPoint, symbol Connector:TestPoint
Connections:
- new net: A1.133 (~{BIOS_SEL}), R2.1, TP78.1
- new net: A1.10 (SIO_UART_TX), J1.1 (Pin_1)
- new net: A1.100 (~{CLKREQ3}), R79.2
- new net: A1.102 (~{CLKREQ4}), R78.2
- new net: A1.12 (SIO_UART_RX), J1.2 (Pin_2)
- new net: A1.185 (TCP1_HPD), R77.1
- new net: A1.187 (TCP0_HPD), R76.1
- new net: BT1.1 (+), R1.1
- new net +BATT: A1.115 (VBAT), R1.2
- new net DDI_B_DDC_SCL: A1.171 (DDIB_DDC_SCL)
- new net DDI_B_DDC_SDA: A1.169 (DDIB_DDC_SDA)
- new net DDI_B_HPD: A1.183 (DDIB_HPD)
- new net DDI_B_TX0+: A1.217 (DDIB_TX0+)
- new net DDI_B_TX0-: A1.215 (DDIB_TX0-)
- new net DDI_B_TX1+: A1.211 (DDIB_TX1+)
- new net DDI_B_TX1-: A1.209 (DDIB_TX1-)
- new net DDI_B_TX2+: A1.205 (DDIB_TX2+)
- new net DDI_B_TX2-: A1.203 (DDIB_TX2-)
- new net DDI_B_TX3+: A1.199 (DDIB_TX3+)
- new net DDI_B_TX3-: A1.197 (DDIB_TX3-)
- new net FAN_1_PWM: A1.2 (FAN1_PWM)
- new net FAN_1_TAC: A1.4 (FAN1_TAC)
- new net GND: A1.101 (GND), A1.107 (GND), A1.11 (GND), A1.110 (GND), A1.113 (GND), A1.116 (GND), A1.135 (GND), A1.136 (GND), A1.14 (GND), A1.151 (GND), A1.158 (GND), A1.167 (GND), A1.17 (GND), A1.170 (GND), A1.181 (GND), A1.182 (GND), A1.188 (GND), A1.189 (GND), A1.194 (GND), A1.195 (GND), A1.20 (GND), A1.200 (GND), A1.201 (GND), A1.206 (GND), A1.207 (GND), A1.212 (GND), A1.213 (GND), A1.218 (GND), A1.219 (GND), A1.224 (GND), A1.225 (GND), A1.23 (GND), A1.230 (GND), A1.231 (GND), A1.236 (GND), A1.237 (GND), A1.242 (GND), A1.243 (GND), A1.248 (GND), A1.249 (GND), A1.26 (GND), A1.29 (GND), A1.32 (GND), A1.35 (GND), A1.38 (GND), A1.41 (GND), A1.44 (GND), A1.47 (GND), A1.50 (GND), A1.53 (GND), A1.56 (GND), A1.59 (GND), A1.62 (GND), A1.65 (GND), A1.68 (GND), A1.71 (GND), A1.74 (GND), A1.77 (GND), A1.80 (GND), A1.83 (GND), A1.86 (GND), A1.89 (GND), A1.92 (GND), A1.95 (GND), A1.98 (GND), A1.MP (Mountinge_Pads), BT1.2 (-), J1.3 (Pin_3), R76.2, R77.2, R78.1, R79.1
- new net GPP_D0: A1.128 (GPP_D0)
- new net GPP_D1: A1.130 (GPP_D1)
- new net GPP_D2: A1.132 (GPP_D2)
- new net GPP_D3: A1.134 (GPP_D3)
- new net HSIO_0_RX+: A1.16 (HSIO0_RX+)
- new net HSIO_0_RX-: A1.18 (HSIO0_RX-)
- new net HSIO_0_TX+: A1.13 (HSIO0_TX+)
- new net HSIO_0_TX-: A1.15 (HSIO0_TX-)
- new net HSIO_10_RX+: A1.52 (HSIO10_RX+)
- new net HSIO_10_RX-: A1.54 (HSIO10_RX-)
- new net HSIO_10_TX+: A1.49 (HSIO10_TX+)
- new net HSIO_10_TX-: A1.51 (HSIO10_TX-)
- new net HSIO_11_RX+: A1.58 (HSIO11_RX+)
- new net HSIO_11_RX-: A1.60 (HSIO11_RX-)
- new net HSIO_11_TX+: A1.55 (HSIO11_TX+)
- new net HSIO_11_TX-: A1.57 (HSIO11_TX-)
- new net HSIO_1_RX+: A1.22 (HSIO1_RX+)
- new net HSIO_1_RX-: A1.24 (HSIO1_RX-)
- new net HSIO_1_TX+: A1.19 (HSIO1_TX+)
- new net HSIO_1_TX-: A1.21 (HSIO1_TX-)
- new net HSIO_2_RX+: A1.28 (HSIO2_RX+)
- new net HSIO_2_RX-: A1.30 (HSIO2_RX-)
- new net HSIO_2_TX+: A1.25 (HSIO2_TX+)
- new net HSIO_2_TX-: A1.27 (HSIO2_TX-)
- new net HSIO_3_RX+: A1.34 (HSIO3_RX+)
- new net HSIO_3_RX-: A1.36 (HSIO3_RX-)
- new net HSIO_3_TX+: A1.31 (HSIO3_TX+)
- new net HSIO_3_TX-: A1.33 (HSIO3_TX-)
- new net HSIO_6_RX+: A1.64 (HSIO6_RX+)
- new net HSIO_6_RX-: A1.66 (HSIO6_RX-)
- new net HSIO_6_TX+: A1.61 (HSIO6_TX+)
- new net HSIO_6_TX-: A1.63 (HSIO6_TX-)
- new net HSIO_8_RX+: A1.40 (HSIO8_RX+)
- new net HSIO_8_RX-: A1.42 (HSIO8_RX-)
- new net HSIO_8_TX+: A1.37 (HSIO8_TX+)
- new net HSIO_8_TX-: A1.39 (HSIO8_TX-)
- new net HSIO_9_RX+: A1.46 (HSIO9_RX+)
- new net HSIO_9_RX-: A1.48 (HSIO9_RX-)
- new net HSIO_9_TX+: A1.43 (HSIO9_TX+)
- new net HSIO_9_TX-: A1.45 (HSIO9_TX-)
- new net I2C2_SCL: A1.154 (I2C2_SCL)
- new net I2C2_SDA: A1.156 (I2C2_SDA)
- new net I2C3_SCL: A1.150 (I2C3_SCL)
- new net I2C3_SDA: A1.152 (I2C3_SDA)
- new net I2C4_SCL: A1.146 (I2C4_SCL)
- new net I2C4_SDA: A1.148 (I2C4_SDA)
- new net I2C5_SCL: A1.142 (I2C5_SCL)
- new net I2C5_SDA: A1.144 (I2C5_SDA)
- new net REFCLK_0+: A1.85 (REFCLK0+)
- new net REFCLK_0-: A1.87 (REFCLK0-)
- new net REFCLK_2+: A1.97 (REFCLK2+)
- new net REFCLK_2-: A1.99 (REFCLK2-)
- new net REFCLK_3+: A1.88 (REFCLK3+)
- new net REFCLK_3-: A1.90 (REFCLK3-)
- new net REFCLK_4+: A1.94 (REFCLK4+)
- new net REFCLK_4-: A1.96 (REFCLK4-)
- new net SLS_S3: A1.7 (SLS_S3)
- new net SOC_UART0_RX: A1.137 (UART0_RXD)
- new net SOC_UART0_TX: A1.139 (UART0_TXD)
- new net SOC_UART1_RX: A1.141 (UART1_RXD)
- new net SOC_UART1_TX: A1.143 (UART1_TXD)
- new net SOC_UART2_RX: A1.140 (UART2_RXD)
- new net SOC_UART2_TX: A1.138 (UART2_TXD)
- new net SUSCLK_WIFI: A1.131 (SUSCLK)
- new net USB_2_P1+: A1.69 (USB2_P1+)
- new net USB_2_P1-: A1.67 (USB2_P1-)
- new net USB_2_P2+: A1.75 (USB2_P2+)
- new net USB_2_P2-: A1.73 (USB2_P2-)
- new net USB_2_P3+: A1.81 (USB2_P3+)
- new net USB_2_P3-: A1.79 (USB2_P3-)
- new net USB_2_P5+: A1.111 (USB2_P5+)
- new net USB_2_P5-: A1.109 (USB2_P5-)
- new net USB_2_P7+: A1.76 (USB2_P7+)
- new net USB_2_P7-: A1.78 (USB2_P7-)
- new net VDC: A1.250 (VIN), A1.251 (VIN), A1.252 (VIN), A1.253 (VIN), A1.254 (VIN), A1.255 (VIN), A1.256 (VIN), A1.257 (VIN), A1.258 (VIN), A1.259 (VIN), A1.260 (VIN)
- new net VPullup: R2.2
- new net ~{PEWAKE}: A1.103 (~{WAKE})
- new net ~{PLT_RST}: A1.105 (~{PLTRST})
- new net ~{PWR_LED}/~{PSON}: A1.5 (SLS_S0)
- new net ~{PWR_SW}: A1.1 (~{PWRBTN})
- new net ~{RST_SW}: A1.3 (~{RSTBTN})
- no-connect marks 0 -> 84
Other:
- note added: "All I2C have integrated pull-up resistors. no need to add pull-up resistors"
- note added: "DDI/TCP functions are defined by the BIOS source code, Cannot be changed in BIOS settings. Before starting design, you should choose one of the available BIOS configurations on: https://github.com/LattePandaTeam/LattePanda-Mu The default functions are defined as follows: - DDIA: eDP 1.4b (the 40Pin connector on the Mu) - DDIB: HDMI 2.0 - TCP0: HDMI 2.0 - TCP1: USB TypeC (need external PD controll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"
- note added: "Debug uart"
- note added: "HPD pin of unused DDI/TCP port needs to be pulled down"
- note added: "HSIO functions are defined by the BIOS source code, Cannot be changed in BIOS settings. Before starting design, you should choose one of the available BIOS configurations on: https://github.com/LattePandaTeam/LattePanda-Mu Or contact techsupport for custom your BIOS The default functions are defined as follows: - HSIO0: USB3.2 10Gbps - HSIO1: USB3.2 10Gbps - HSIO2: PCIe 3.0 x1 - HSIO3: PCIe 3.0 x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"
- note added: "Sleeping State Signal - SLS_S0: - S0 (Working): HIGH - S3 (Slpeeping): LOW - S4 (Hibernation): LOW - S5 (Soft Off): LOW - SLS_S3: - S0 (Working): HIGH - S3 (Slpeeping): HIGH - S4 (Hibernation): LOW - S5 (Soft Off): LOW"
- note added: "~{CLKREQ} is reserved for PCIe ASPM L1s Unless the device clearly supports it, pull it down to enhance compatibility"

Commit message: fix: Set missing footprints and fixed missing pin-pad connections.
- J15, J16 missing MP1 and MP2 pins. Fixed in pin table within the symbol editor for each symbol.
- A ll USB receptacles J4, J5, J18 had mismatched pin numbers for the pcb symbol footprint. Renamed to match.
- Fixed various DNP components that were not excluded from the board.
- Fixed remaining missing footprints.
Parts:
- added H5, H6: MountingHole_Pad, A_HDJ_Library:MountingHole_3mm_M2_Pad_TopOnly, symbol Mechanical:MountingHole_Pad
- BT1: footprint (none) -> A_HDJ_Library:Battery_Holder_CR1220_S8411-45R
- R1, R2, R76, R77, R78, R79: footprint (none) -> A_HDJ_Library:R_0402_1005Metric
- TP78: footprint (none) -> A_HDJ_Library:TestPoint_Pad_D1.5mm
Connections:
- net GND: now also H5.1, H6.1
