File: usb_2_3.kicad_sch (KiCad schematic)
At the start: 0 parts

Commit message: feat(usb): Added usb 2.0 & usb 3.0 implementation and connections.
Parts:
- added C26, C27, C29: 100nF/50V, A_HDJ_Library:C_0402_1005Metric, symbol Device:C
- added C30, C31, C32: 22uF/10V, A_HDJ_Library:C_0603_1608Metric, symbol Device:C
- added D5, D6, D7, D8: ESD5V0B03, A_HDJ_Library:D_0402_1005Metric, symbol Diode:ESD9B5.0ST5G
- added F2, F3, F4, F5: 6V/1A, A_HDJ_Library:Fuse_0805_2012Metric, symbol Device:Fuse
- added J4: USB3_A_Stacked, A_HDJ_Library:USB3_A_Molex_48406-0001_Horizontal_Stacked, symbol Connector:USB3_A_Stacked
- added J5: USB_A_Stacked, A_HDJ_Library:USB_A_CUI_UJ2-ADH-TH_Horizontal_Stacked, symbol Connector:USB_A_Stacked
- added U3, U4, U5: D3V3XA4B10LP, A_HDJ_Library:Diodes_UDFN-10_1.0x2.5mm_P0.5mm, symbol Power_Protection:D3V3XA4B10LP
Connections:
- new net: F2.2, J5.1 (VBUS1)
- new net: F5.2, J4.10 (VBUS2)
- new net: F3.2, J5.5 (VBUS2)
- new net: F4.2, J4.1 (VBUS1)
- new net +5V: C30.2, C31.2, C32.2, F2.1, F3.1, F4.1, F5.1
- new net CON_USB3_SSTX_N: C26.2, J4.8 (SSTX1-), U3.4, U3.7 (NC)
- new net CON_USB3_SSTX_P: C27.2, J4.9 (SSTX1+), U3.5, U3.6 (NC)
- new net CON_USB4_SSTX_N: C26.2, J4.17 (SSTX2-), U3.1, U3.10 (NC)
- new net CON_USB4_SSTX_P: C29.2, J4.18 (SSTX2+), U3.2, U3.9 (NC)
- new net GND: C30.1, C31.1, C32.1, D5.2 (A2), D6.2 (A2), D7.2 (A2), D8.2 (A2), J4.13 (GND2), J4.16 (DRAIN2), J4.4 (GND1), J4.7 (DRAIN1), J4.SH (SHIELD), J4.SH (SHIELD), J5.4 (GND1), J5.8 (GND2), J5.SH (Shield), U3.3 (VSS), U3.8 (VSS), U4.3 (VSS), U4.8 (VSS), U5.3 (VSS), U5.8 (VSS)
- new net USB3_SSRX_N: J4.5 (SSRX1-), U5.4, U5.7 (NC)
- new net USB3_SSRX_P: J4.6 (SSRX1+), U5.5, U5.6 (NC)
- new net USB3_SSTX_N: C26.1
- new net USB3_SSTX_P: C27.1
- new net USB4_SSRX_N: J4.14 (SSRX2-), U5.1, U5.10 (NC)
- new net USB4_SSRX_P: J4.15 (SSRX2+), U5.2, U5.9 (NC)
- new net USB4_SSTX_N: C26.1
- new net USB4_SSTX_P: C29.1
- new net USB_2_P1+: D5.1 (A1), J4.12 (D2+)
- new net USB_2_P1-: D6.1 (A1), J4.11 (D2-)
- new net USB_2_P2+: D7.1 (A1), J4.3 (D1+)
- new net USB_2_P2-: D8.1 (A1), J4.2 (D1-)
- new net USB_2_P3+: J5.7 (D2+), U4.4, U4.7 (NC)
- new net USB_2_P3-: J5.6 (D2-), U4.5, U4.6 (NC)
- new net USB_2_P5+: J5.3 (D1+), U4.1, U4.10 (NC)
- new net USB_2_P5-: J5.2 (D1-), U4.2, U4.9 (NC)
Other:
- note added: "USB 2.0"
- note added: "USB 3.0"
- title: (none) -> USB 2.0 & USB 3.0

Commit message: feat(hdmi): Added HDMI implementation and connections.
Parts:
- renumbered C26 to C28
Other:
- moved on the sheet: C26
Changed lines of the file:
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@@
+	(symbol
+		(lib_id "Device:C")
+		(at 181.61 71.12 90)
+		(unit 1)
+		(body_style 1)
+		(exclude_from_sim no)
+		(in_bom yes)
+		(on_board yes)
+		(in_pos_files yes)
+		(dnp no)
+		(property "Reference" "C26"
+			(at 176.53 70.104 90)
+			(show_name no)
+			(do_not_autoplace no)
+			(effects
+				(font
+					(size 1.27 1.27)
+				)
+			)
+		)
+		(property "Value" "100nF/50V"
+			(at 189.738 70.104 90)
+			(show_name no)
+			(do_not_autoplace no)
+			(effects
+				(font
+					(size 1.27 1.27)
+				)
+			)
+		)
+		(property "Footprint" "A_HDJ_Library:C_0402_1005Metric"
+			(at 185.42 70.1548 0)
+			(hide yes)
+			(show_name no)
+			(do_not_autoplace no)
+			(effects
+				(font
+					(size 1.27 1.27)
+				)
+			)
+		)
+		(property "Datasheet" ""
+			(at 181.61 71.12 0)
+			(hide yes)
+			(show_name no)
+			(do_not_autoplace no)
+			(effects
+				(font
+					(size 1.27 1.27)
+				)
+			)
+		)
+		(property "Description" "Unpolarized capacitor"
+			(at 181.61 71.12 0)
+			(hide yes)
+			(show_name no)
+			(do_not_autoplace no)
+			(effects
+				(font
+					(size 1.27 1.27)
+				)
+			)
+		)
+		(pin "1"
+		)
+		(pin "2"
+		)
+		(instances
+			(project "LattePandaMu-Carrier"
+				(path "/07ab76aa-21ac-4dd9-9287-fe7c28981c17/abcea79a-a9ee-4f84-85fd-ba1001f6eea1"
+					(reference "C26")
+					(unit 1)
+				)
+			)
+		)
+	)
 	(symbol
 		(lib_id "Device:C")
@@
 					(unit 1)
 				)
-			)
-		)
-	)
-	(symbol
-		(lib_id "Device:C")
-		(at 181.61 71.12 90)
-		(unit 1)
-		(body_style 1)
-		(exclude_from_sim no)
-		(in_bom yes)
-		(on_board yes)
-		(in_pos_files yes)
-		(dnp no)
-		(property "Reference" "C26"
-			(at 176.53 70.104 90)
-			(show_name no)
-			(do_not_autoplace no)
-			(effects
-				(font
-					(size 1.27 1.27)
-				)
-			)
-		)
-		(property "Value" "100nF/50V"
-			(at 189.738 70.104 90)
-			(show_name no)
-			(do_not_autoplace no)
-			(effects
-				(font
-					(size 1.27 1.27)
-				)
-			)
-		)
-		(property "Footprint" "A_HDJ_Library:C_0402_1005Metric"
-			(at 185.42 70.1548 0)
-			(hide yes)
-			(show_name no)
-			(do_not_autoplace no)
-			(effects
-				(font
-					(size 1.27 1.27)
-				)
-			)
-		)
-		(property "Datasheet" ""
-			(at 181.61 71.12 0)
-			(hide yes)
-			(show_name no)
-			(do_not_autoplace no)
-			(effects
-				(font
-					(size 1.27 1.27)
-				)
-			)
-		)
-		(property "Description" "Unpolarized capacitor"
-			(at 181.61 71.12 0)
-			(hide yes)
-			(show_name no)
-			(do_not_autoplace no)
-			(effects
-				(font
-					(size 1.27 1.27)
-				)
-			)
-		)
-		(pin "1"
-		)
-		(pin "2"
-		)
-		(instances
-			(project "LattePandaMu-Carrier"
-				(path "/07ab76aa-21ac-4dd9-9287-fe7c28981c17/abcea79a-a9ee-4f84-85fd-ba1001f6eea1"
-					(reference "C26")
-					(unit 1)
-				)

Commit message: fix: Set missing footprints and fixed missing pin-pad connections.
- J15, J16 missing MP1 and MP2 pins. Fixed in pin table within the symbol editor for each symbol.
- A ll USB receptacles J4, J5, J18 had mismatched pin numbers for the pcb symbol footprint. Renamed to match.
- Fixed various DNP components that were not excluded from the board.
- Fixed remaining missing footprints.
Parts:
- added C28: 100nF/50V, A_HDJ_Library:C_0402_1005Metric, symbol Device:C
- renumbered C28 to C26
Connections:
- net CON_USB4_SSTX_N: now also C28.2; no longer C26.2
- net GND: now also J4.19 (SHIELD), J4.19 (SHIELD), J5.9 (Shield); no longer J4.SH (SHIELD), J4.SH (SHIELD), J5.SH (Shield)
- net USB4_SSTX_N: now also C28.1; no longer C26.1
