File: fan.kicad_sch (KiCad schematic)
At the start: 0 parts

Commit message: feat(fan): Added fan circuit and connected sheet pins
Parts:
- added C84, C85: 100nF/50V, A_HDJ_Library:C_0402_1005Metric, symbol Device:C
- added D26, D27: 1N5819WS, A_HDJ_Library:D_SOD-323, symbol Diode:1N5819WS
- added JP2: NTC_Test, Jumper:SolderJumper-2_P1.3mm_Open_RoundedPad1.0x1.5mm, symbol Jumper:SolderJumper_2_Open
- added M1, M2: Fan_4pin, A_HDJ_Library:JST_PH_B4B-PH-K_1x04_P2.00mm_Vertical, symbol Motor:Fan_4pin
- added R63: 10k/1%, A_HDJ_Library:R_0402_1005Metric, symbol Device:R
- added R64, R65, R72, R74: 4.7k/1%, A_HDJ_Library:R_0402_1005Metric, symbol Device:R
- added R66, R67, R68, R70: 21.5k/1%, A_HDJ_Library:R_0402_1005Metric, symbol Device:R
- added R69, R71: 100R/1%, A_HDJ_Library:R_0402_1005Metric, symbol Device:R
- added R73, R75: 0R/1%, RES0603, symbol Device:R
- added TH1: NTC-10K, Resistor_SMD:R_0603_1608Metric, symbol Device:Thermistor_NTC
- added TP11, TP12: TestPoint, symbol Connector:TestPoint
Connections:
- new net: JP2.2 (B), R63.2, TH1.1
- new net: M1.4 (PWM), R69.2
- new net: D27.2 (A), M2.3 (Tacho), R70.2, R74.2
- new net: D26.2 (A), M1.3 (Tacho), R68.2, R72.2
- new net: C85.1, D27.1 (K), M2.2 (+), R73.2, R74.1, R75.2
- new net: M2.4 (PWM), R71.2
- new net +12V: R75.1
- new net +3.3V: R63.1, R64.1, R65.1
- new net +5V: C84.1, D26.1 (K), M1.2 (+), R72.1, R73.1
- new net FAN_1_PWM: R64.2, R69.1, TP12.1
- new net FAN_1_TAC: R66.1, R68.1, TP11.1
- new net FAN_2_PWM: R65.2, R71.1
- new net FAN_2_TAC: R67.1, R70.1
- new net GND: C84.2, C85.2, M1.1 (-), M2.1 (-), R66.2, R67.2, TH1.2
- new net TEMP: JP2.1 (A)
Other:
- note added: "CPU FAN"
- note added: "LattePanda Mu has integrated pull-up resistors."
- note added: "Reserved for 12V fan FAN_TAC input only allows 3.3V level"
- note added: "SYS FAN"
- note added: "TEMP"

Commit message: fix: Set missing footprints and fixed missing pin-pad connections.
- J15, J16 missing MP1 and MP2 pins. Fixed in pin table within the symbol editor for each symbol.
- A ll USB receptacles J4, J5, J18 had mismatched pin numbers for the pcb symbol footprint. Renamed to match.
- Fixed various DNP components that were not excluded from the board.
- Fixed remaining missing footprints.
Parts:
- R73, R75: now left out of the parts list
- TP11, TP12: footprint (none) -> A_HDJ_Library:TestPoint_Pad_D1.5mm

Commit message: fix: Fixed DNP parts populating on the board.
Parts:
- C85, D27, M2, R63, R64, R65, R66, R67, R70, R71, R74: now left out of the parts list
Changed lines of the file:
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@@
 		(body_style 1)
 		(exclude_from_sim no)
-		(in_bom yes)
-		(on_board yes)
+		(in_bom no)
+		(on_board no)
 		(in_pos_files yes)
 		(dnp yes)
@@
 		(body_style 1)
 		(exclude_from_sim no)
-		(in_bom yes)
-		(on_board yes)
+		(in_bom no)
+		(on_board no)
 		(in_pos_files yes)
 		(dnp yes)
@@
 		(body_style 1)
 		(exclude_from_sim no)
-		(in_bom yes)
-		(on_board yes)
+		(in_bom no)
+		(on_board no)
 		(in_pos_files yes)
 		(dnp yes)
@@
 		(body_style 1)
 		(exclude_from_sim no)
-		(in_bom yes)
-		(on_board yes)
+		(in_bom no)
+		(on_board no)
 		(in_pos_files yes)
 		(dnp yes)
@@
 		(body_style 1)
 		(exclude_from_sim no)
-		(in_bom yes)
-		(on_board yes)
+		(in_bom no)
+		(on_board no)
 		(in_pos_files yes)
 		(dnp yes)
@@
 		(body_style 1)
 		(exclude_from_sim no)
-		(in_bom yes)
-		(on_board yes)
+		(in_bom no)
+		(on_board no)
 		(in_pos_files yes)
 		(dnp yes)
@@
 		(body_style 1)
 		(exclude_from_sim no)
-		(in_bom yes)
-		(on_board yes)
+		(in_bom no)
+		(on_board no)
 		(in_pos_files yes)
 		(dnp yes)
@@
 		(body_style 1)
 		(exclude_from_sim no)
-		(in_bom yes)
-		(on_board yes)
+		(in_bom no)
+		(on_board no)
 		(in_pos_files yes)
 		(dnp yes)
@@
 		(body_style 1)
 		(exclude_from_sim no)
-		(in_bom yes)
-		(on_board yes)
+		(in_bom no)
+		(on_board no)
 		(in_pos_files yes)
 		(dnp yes)
@@
 		(body_style 1)
 		(exclude_from_sim no)
-		(in_bom yes)
-		(on_board yes)
+		(in_bom no)
+		(on_board no)
 		(in_pos_files yes)
 		(dnp yes)
@@
 		(body_style 1)
 		(exclude_from_sim no)
-		(in_bom yes)
-		(on_board yes)
+		(in_bom no)
+		(on_board no)
 		(in_pos_files yes)
 		(dnp yes)
