File: picex4.kicad_sch (KiCad schematic)
At the start: 0 parts

Commit message: feat(pcie): Added PCIe x4 implementation and connections.
Parts:
- added C1, C2, C3, C4, C5, C6, C7, C8: 220nF/50V, A_HDJ_Library:C_0402_1005Metric, symbol Device:C_Small
- added C10, C13, C15, C9: 100nF/50V, A_HDJ_Library:C_0402_1005Metric, symbol Device:C
- added C11: 100uF/25V, A_HDJ_Library:CP_Elec_6.3x7.7, symbol Device:C_Polarized
- added C14: 10uF/10V, A_HDJ_Library:C_0402_1005Metric, symbol Device:C
- added C16: 560uF/25V, A_HDJ_Library:CP_Elec_6.3x7.7, symbol Device:C_Polarized
- added J2: Bus_PCI_Express_x4, A_HDJ_Library:PCIe_x4_Gen3Slot_Connectors, symbol Connector:Bus_PCI_Express_x4
Connections:
- new net +12VA: C10.1, C11.1, C9.1, J2.A2 (+12V), J2.A3 (+12V), J2.B1 (+12V), J2.B2 (+12V), J2.B3 (+12V)
- new net +3.3V: C13.2, C14.2, C15.1, C16.1, J2.A10 (+3.3V), J2.A9 (+3.3V), J2.B10 (3.3Vaux), J2.B8 (+3.3V)
- new net GND: C10.2, C11.2, C13.1, C14.1, C15.2, C16.2, C9.2, J2.A1 (~{PRSNT1}), J2.A12 (GND), J2.A15 (GND), J2.A18 (GND), J2.A20 (GND), J2.A23 (GND), J2.A24 (GND), J2.A27 (GND), J2.A28 (GND), J2.A31 (GND), J2.A4 (GND), J2.B13 (GND), J2.B16 (GND), J2.B17 (~{PRSNT2}), J2.B18 (GND), J2.B21 (GND), J2.B22 (GND), J2.B25 (GND), J2.B26 (GND), J2.B29 (GND), J2.B31 (~{PRSNT2}), J2.B32 (GND), J2.B4 (GND), J2.B7 (GND)
- new net PCIE30_TX0_N: C2.2, J2.B15 (PETn0)
- new net PCIE30_TX0_P: C1.2, J2.B14 (PETp0)
- new net PCIE30_TX1_N: C4.2, J2.B20 (PETn1)
- new net PCIE30_TX1_P: C3.2, J2.B19 (PETp1)
- new net PCIE30_TX2_N: C6.2, J2.B24 (PETn2)
- new net PCIE30_TX2_P: C5.2, J2.B23 (PETp2)
- new net PCIE30_TX3_N: C8.2, J2.B28 (PETn3)
- new net PCIE30_TX3_P: C7.2, J2.B27 (PETp3)
- new net PCIE_RX_0+: J2.A16 (PERp0)
- new net PCIE_RX_0-: J2.A17 (PERn0)
- new net PCIE_RX_1+: J2.A21 (PERp1)
- new net PCIE_RX_1-: J2.A22 (PERn1)
- new net PCIE_RX_2+: J2.A25 (PERp2)
- new net PCIE_RX_2-: J2.A26 (PERn2)
- new net PCIE_RX_3+: J2.A29 (PERp3)
- new net PCIE_RX_3-: J2.A30 (PERn3)
- new net PCIE_TX_0+: C1.1
- new net PCIE_TX_0-: C2.1
- new net PCIE_TX_1+: C3.1
- new net PCIE_TX_1-: C4.1
- new net PCIE_TX_2+: C5.1
- new net PCIE_TX_2-: C6.1
- new net PCIE_TX_3+: C7.1
- new net PCIE_TX_3-: C8.1
- new net REFCLK+: J2.A13 (REFCLK+)
- new net REFCLK-: J2.A14 (REFCLK-)
- new net ~{PR_RST}: J2.A11 (~{PERST})
- new net ~{WAKE}: J2.B11 (~{WAKE})
- no-connect marks 0 -> 11

Commit message: fix: Fixed DNP parts populating on the board.
Parts:
- C1, C10, C11, C13, C14, C15, C16, C2, C3, C4, C5, C6, C7, C8, C9, J2: now left out of the parts list
Changed lines of the file:
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@@
 		(body_style 1)
 		(exclude_from_sim no)
-		(in_bom yes)
-		(on_board yes)
+		(in_bom no)
+		(on_board no)
 		(in_pos_files yes)
 		(dnp yes)
@@
 		(body_style 1)
 		(exclude_from_sim no)
-		(in_bom yes)
-		(on_board yes)
+		(in_bom no)
+		(on_board no)
 		(in_pos_files yes)
 		(dnp yes)
@@
 		(body_style 1)
 		(exclude_from_sim no)
-		(in_bom yes)
-		(on_board yes)
+		(in_bom no)
+		(on_board no)
 		(in_pos_files yes)
 		(dnp yes)
@@
 		(body_style 1)
 		(exclude_from_sim no)
-		(in_bom yes)
-		(on_board yes)
+		(in_bom no)
+		(on_board no)
 		(in_pos_files yes)
 		(dnp yes)
@@
 		(body_style 1)
 		(exclude_from_sim no)
-		(in_bom yes)
-		(on_board yes)
+		(in_bom no)
+		(on_board no)
 		(in_pos_files yes)
 		(dnp yes)
@@
 		(body_style 1)
 		(exclude_from_sim no)
-		(in_bom yes)
-		(on_board yes)
+		(in_bom no)
+		(on_board no)
 		(in_pos_files yes)
 		(dnp yes)
@@
 		(body_style 1)
 		(exclude_from_sim no)
-		(in_bom yes)
-		(on_board yes)
+		(in_bom no)
+		(on_board no)
 		(in_pos_files yes)
 		(dnp yes)
@@
 		(body_style 1)
 		(exclude_from_sim no)
-		(in_bom yes)
-		(on_board yes)
+		(in_bom no)
+		(on_board no)
 		(in_pos_files yes)
 		(dnp yes)
@@
 		(body_style 1)
 		(exclude_from_sim no)
-		(in_bom yes)
-		(on_board yes)
+		(in_bom no)
+		(on_board no)
 		(in_pos_files yes)
 		(dnp yes)
@@
 		(body_style 1)
 		(exclude_from_sim no)
-		(in_bom yes)
-		(on_board yes)
+		(in_bom no)
+		(on_board no)
 		(in_pos_files yes)
 		(dnp yes)
@@
 		(body_style 1)
 		(exclude_from_sim no)
-		(in_bom yes)
-		(on_board yes)
+		(in_bom no)
+		(on_board no)
 		(in_pos_files yes)
 		(dnp yes)
@@
 		(body_style 1)
 		(exclude_from_sim no)
-		(in_bom yes)
-		(on_board yes)
+		(in_bom no)
+		(on_board no)
 		(in_pos_files yes)
 		(dnp yes)
@@
 		(body_style 1)
 		(exclude_from_sim no)
-		(in_bom yes)
-		(on_board yes)
+		(in_bom no)
+		(on_board no)
 		(in_pos_files yes)
 		(dnp yes)
@@
 		(body_style 1)
 		(exclude_from_sim no)
-		(in_bom yes)
-		(on_board yes)
+		(in_bom no)
+		(on_board no)
 		(in_pos_files yes)
 		(dnp yes)
@@
 		(body_style 1)
 		(exclude_from_sim no)
-		(in_bom yes)
-		(on_board yes)
+		(in_bom no)
+		(on_board no)
 		(in_pos_files yes)
 		(dnp yes)
@@
 		(body_style 1)
 		(exclude_from_sim no)
-		(in_bom yes)
-		(on_board yes)
+		(in_bom no)
+		(on_board no)
 		(in_pos_files yes)
 		(dnp yes)
@@
 		(body_style 1)
 		(exclude_from_sim no)
-		(in_bom yes)
-		(on_board yes)
+		(in_bom no)
+		(on_board no)
 		(in_pos_files yes)
 		(dnp yes)
@@
 		(body_style 1)
 		(exclude_from_sim no)
-		(in_bom yes)
-		(on_board yes)
+		(in_bom no)
+		(on_board no)
 		(in_pos_files yes)
 		(dnp yes)
@@
 		(body_style 1)
 		(exclude_from_sim no)
-		(in_bom yes)
-		(on_board yes)
+		(in_bom no)
+		(on_board no)
 		(in_pos_files yes)
 		(dnp yes)
@@
 		(body_style 1)
 		(exclude_from_sim no)
-		(in_bom yes)
-		(on_board yes)
+		(in_bom no)
+		(on_board no)
 		(in_pos_files yes)
 		(dnp yes)
@@
 		(body_style 1)
 		(exclude_from_sim no)
-		(in_bom yes)
-		(on_board yes)
+		(in_bom no)
+		(on_board no)
 		(in_pos_files yes)
 		(dnp yes)
@@
 		(body_style 1)
 		(exclude_from_sim no)
-		(in_bom yes)
-		(on_board yes)
+		(in_bom no)
+		(on_board no)
 		(in_pos_files yes)
 		(dnp yes)
@@
 		(body_style 1)
 		(exclude_from_sim no)
-		(in_bom yes)
-		(on_board yes)
-		(in_pos_files yes)
-		(dnp yes)
+		(in_bom no)
+		(on_board no)
+		(in_pos_files yes)
+		(dnp yes)
