File: LattePandaMu-Carrier.kicad_pcb (KiCad board)
At the start: 4 copper layers, 0 parts

Commit message: feat(pcb): Board outline and import
Parts:
- added A1: LattePanda_Mu, Module_LattePanda:LattePanda_Module_H8.0mm_Horizontal, F.Cu at (342.7, 34.2)
- added C1: 220nF/50V, A_HDJ_Library:C_0402_1005Metric, F.Cu at (395.8, 41.5)
- added C10: 100nF/50V, A_HDJ_Library:C_0402_1005Metric, F.Cu at (398.7, 49.4)
- added C11: 100uF/25V, A_HDJ_Library:CP_Elec_6.3x7.7, F.Cu at (389.2, 44.6)
- added C13: 100nF/50V, A_HDJ_Library:C_0402_1005Metric, F.Cu at (401.6, 41.5)
- added C14: 10uF/10V, A_HDJ_Library:C_0402_1005Metric, F.Cu at (401.6, 43.5)
- added C15: 100nF/50V, A_HDJ_Library:C_0402_1005Metric, F.Cu at (401.6, 45.5)
- added C16: 560uF/25V, A_HDJ_Library:CP_Elec_6.3x7.7, F.Cu at (389.2, 52.8)
- added C17: 100nF/50V, A_HDJ_Library:C_0402_1005Metric, F.Cu at (384.0, 149.6)
- added C18: 100nF/50V, A_HDJ_Library:C_0402_1005Metric, F.Cu at (384.0, 151.5)
- added C19: 100nF/50V, A_HDJ_Library:C_0402_1005Metric, F.Cu at (384.0, 153.5)
- added C2: 220nF/50V, A_HDJ_Library:C_0402_1005Metric, F.Cu at (395.8, 43.5)
- added C20: 100nF/50V, A_HDJ_Library:C_0402_1005Metric, F.Cu at (386.9, 149.6)
- added C21: 100nF/50V, A_HDJ_Library:C_0402_1005Metric, F.Cu at (386.9, 151.5)
- added C22: 100nF/50V, A_HDJ_Library:C_0402_1005Metric, F.Cu at (386.9, 153.5)
- added C23: 100nF/50V, A_HDJ_Library:C_0402_1005Metric, F.Cu at (389.8, 149.6)
- added C24: 100nF/50V, A_HDJ_Library:C_0402_1005Metric, F.Cu at (389.8, 151.5)
- added C25: 100nF/50V, A_HDJ_Library:C_0402_1005Metric, F.Cu at (389.8, 153.5)
- added C26: 100nF/50V, A_HDJ_Library:C_0402_1005Metric, F.Cu at (324.7, 107.6)
- added C27: 100nF/50V, A_HDJ_Library:C_0402_1005Metric, F.Cu at (324.7, 109.6)
- added C28: 100nF/50V, A_HDJ_Library:C_0402_1005Metric, F.Cu at (324.7, 111.6)
- added C29: 100nF/50V, A_HDJ_Library:C_0402_1005Metric, F.Cu at (324.7, 113.5)
- added C3: 220nF/50V, A_HDJ_Library:C_0402_1005Metric, F.Cu at (395.8, 45.5)
- added C30: 22uF/10V, A_HDJ_Library:C_0603_1608Metric, F.Cu at (328.2, 107.9)
- added C31: 22uF/10V, A_HDJ_Library:C_0603_1608Metric, F.Cu at (328.2, 110.4)
- added C32: 22uF/10V, A_HDJ_Library:C_0603_1608Metric, F.Cu at (328.2, 112.9)
- added C33: 100nF/50V, A_HDJ_Library:C_0402_1005Metric, F.Cu at (419.1, 107.6)
- added C34: 100nF/50V, A_HDJ_Library:C_0402_1005Metric, F.Cu at (419.1, 109.6)
- added C35: 100nF/50V, A_HDJ_Library:C_0402_1005Metric, F.Cu at (419.1, 111.6)
- added C37: 100nF/50V, A_HDJ_Library:C_0402_1005Metric, F.Cu at (419.1, 113.5)
- added C38: 100nF/50V, A_HDJ_Library:C_0402_1005Metric, F.Cu at (419.1, 115.5)
- added C39: 100nF/50V, A_HDJ_Library:C_0402_1005Metric, F.Cu at (419.1, 117.5)
- added C4: 220nF/50V, A_HDJ_Library:C_0402_1005Metric, F.Cu at (395.8, 47.4)
- added C40: 100nF/50V, A_HDJ_Library:C_0402_1005Metric, F.Cu at (422.0, 107.6)
- added C41: 100nF/50V, A_HDJ_Library:C_0402_1005Metric, F.Cu at (422.0, 109.6)
- added C42: 100nF/50V, A_HDJ_Library:C_0402_1005Metric, F.Cu at (422.0, 111.6)
- added C43: 100nF/50V, A_HDJ_Library:C_0402_1005Metric, F.Cu at (422.0, 113.5)
- added C44: 10uF/50V, A_HDJ_Library:C_0402_1005Metric, F.Cu at (422.0, 115.5)
- added C45: 100nF/50V, A_HDJ_Library:C_0402_1005Metric, F.Cu at (422.0, 117.5)
- added C46: 12pF/50V, A_HDJ_Library:C_0402_1005Metric, F.Cu at (424.9, 107.6)
- added C47: 12pF/50V, A_HDJ_Library:C_0402_1005Metric, F.Cu at (424.9, 109.6)
- added C48: 100nF/50V, A_HDJ_Library:C_0402_1005Metric, F.Cu at (424.9, 111.6)
- added C49: 220nF/50V, A_HDJ_Library:C_0402_1005Metric, F.Cu at (337.4, 132.6)
- added C5: 220nF/50V, A_HDJ_Library:C_0402_1005Metric, F.Cu at (395.8, 49.4)
- added C50: 220nF/50V, A_HDJ_Library:C_0402_1005Metric, F.Cu at (337.4, 134.6)
- added C51: 100nF/50V, A_HDJ_Library:C_0402_1005Metric, F.Cu at (337.4, 136.5)
- added C52: 100nF/50V, A_HDJ_Library:C_0402_1005Metric, F.Cu at (337.4, 138.5)
- added C53: 100nF/50V, A_HDJ_Library:C_0402_1005Metric, F.Cu at (340.3, 132.6)
- added C54: 100nF/50V, A_HDJ_Library:C_0402_1005Metric, F.Cu at (340.3, 134.6)
- added C55: 220nF/50V, A_HDJ_Library:C_0402_1005Metric, F.Cu at (340.3, 136.5)
- added C56: 220nF/50V, A_HDJ_Library:C_0402_1005Metric, F.Cu at (340.3, 138.5)
- added C57: 100nF/50V, A_HDJ_Library:C_0402_1005Metric, F.Cu at (343.1, 132.6)
- added C58: 100nF/50V, A_HDJ_Library:C_0402_1005Metric, F.Cu at (343.1, 134.6)
- added C59: 100nF/50V, A_HDJ_Library:C_0402_1005Metric, F.Cu at (343.1, 136.5)
- added C6: 220nF/50V, A_HDJ_Library:C_0402_1005Metric, F.Cu at (398.7, 41.5)
- added C60: 100nF/50V, A_HDJ_Library:C_0402_1005Metric, F.Cu at (343.1, 138.5)
- added C61: 1uF/16V, A_HDJ_Library:C_0402_1005Metric, F.Cu at (421.4, 74.9)
- added C62: 1uF/16V, A_HDJ_Library:C_0402_1005Metric, F.Cu at (421.4, 76.9)
- added C63: 1uF/16V, A_HDJ_Library:C_0402_1005Metric, F.Cu at (421.4, 78.8)
- added C64: 22uF/10V, A_HDJ_Library:C_0603_1608Metric, F.Cu at (398.9, 60.1)
- added C65: 22uF/10V, A_HDJ_Library:C_0603_1608Metric, F.Cu at (398.9, 62.6)
- added C66: 1uF/16V, A_HDJ_Library:C_0402_1005Metric, F.Cu at (421.4, 80.8)
- added C67: 22uF/10V, A_HDJ_Library:C_0603_1608Metric, F.Cu at (398.9, 65.1)
- added C68: 22uF/10V, A_HDJ_Library:C_0603_1608Metric, F.Cu at (398.9, 67.6)
- added C69: 1uF/16V, A_HDJ_Library:C_0402_1005Metric, F.Cu at (421.4, 82.8)
- added C7: 220nF/50V, A_HDJ_Library:C_0402_1005Metric, F.Cu at (398.7, 43.5)
- added C70: 100nF/50V, A_HDJ_Library:C_0603_1608Metric, F.Cu at (398.9, 70.1)
- added C71: 100nF/50V, A_HDJ_Library:C_0603_1608Metric, F.Cu at (398.9, 72.7)
- added C72: 12pF/50V, A_HDJ_Library:C_0402_1005Metric, F.Cu at (421.4, 84.7)
- added C73: 12pF/50V, A_HDJ_Library:C_0402_1005Metric, F.Cu at (421.4, 86.7)
- added C74: 22uF/10V, A_HDJ_Library:C_0603_1608Metric, F.Cu at (402.9, 60.1)
- added C75: 22uF/10V, A_HDJ_Library:C_0603_1608Metric, F.Cu at (402.9, 62.6)
- added C76: 22uF/10V, A_HDJ_Library:C_0603_1608Metric, F.Cu at (402.9, 65.1)
- added C77: 22uF/10V, A_HDJ_Library:C_0603_1608Metric, F.Cu at (402.9, 67.6)
- added C78: 100nF/50V, A_HDJ_Library:C_0603_1608Metric, F.Cu at (402.9, 70.1)
- added C79: 100nF/50V, A_HDJ_Library:C_0603_1608Metric, F.Cu at (402.9, 72.7)
- added C8: 220nF/50V, A_HDJ_Library:C_0402_1005Metric, F.Cu at (398.7, 45.5)
- added C80: 22uF/10V, A_HDJ_Library:C_0603_1608Metric, F.Cu at (407.0, 60.1)
- added C81: 22uF/10V, A_HDJ_Library:C_0603_1608Metric, F.Cu at (407.0, 62.6)
- added C82: 22uF/10V, A_HDJ_Library:C_0603_1608Metric, F.Cu at (407.0, 65.1)
- added C83: 22uF/10V, A_HDJ_Library:C_0603_1608Metric, F.Cu at (407.0, 67.6)
- added C84: 100nF/50V, A_HDJ_Library:C_0402_1005Metric, F.Cu at (399.0, 150.8)
- added C85: 100nF/50V, A_HDJ_Library:C_0402_1005Metric, F.Cu at (399.0, 152.7)
- added C9: 100nF/50V, A_HDJ_Library:C_0402_1005Metric, F.Cu at (398.7, 47.4)
- added D1: ESD5V0B03, A_HDJ_Library:D_0402_1005Metric, F.Cu at (384.1, 135.6)
- added D10: ESD9B5.0ST5G, A_HDJ_Library:D_0402_1005Metric, F.Cu at (410.4, 59.8)
- added D11: ESD9B5.0ST5G, A_HDJ_Library:D_0402_1005Metric, F.Cu at (410.4, 61.8)
- added D12: D_Zener, A_HDJ_Library:D_0402_1005Metric, F.Cu at (410.4, 63.8)
- added D13: D_Zener, A_HDJ_Library:D_0402_1005Metric, F.Cu at (410.4, 65.8)
- added D14: D_Zener, A_HDJ_Library:D_0402_1005Metric, F.Cu at (410.4, 67.8)
- added D15: D_Schottky, A_HDJ_Library:D_SMA, F.Cu at (388.0, 61.1)
- added D16: D_Schottky, A_HDJ_Library:D_SMA, F.Cu at (388.0, 65.7)
- added D17: D_Schottky, A_HDJ_Library:D_SMA, F.Cu at (388.0, 70.2)
- added D18: D_Schottky, A_HDJ_Library:D_SMA, F.Cu at (388.0, 74.8)
- added D19: D_Schottky, A_HDJ_Library:D_SMA, F.Cu at (388.0, 79.3)
- added D2: ESD5V0B03, A_HDJ_Library:D_0402_1005Metric, F.Cu at (384.1, 137.6)
- added D20: D_Schottky, A_HDJ_Library:D_SMA, F.Cu at (388.0, 83.9)
- added D21: ESD9B5.0ST5G, Diode_SMD:D_0402_1005Metric, F.Cu at (393.7, 77.6)
- added D22: LED, A_HDJ_Library:LED_0603_1608Metric, F.Cu at (405.3, 89.6)
- added D23: LED, A_HDJ_Library:LED_0603_1608Metric, F.Cu at (405.3, 92.1)
- added D24: 3V3 Izt=5mA, A_HDJ_Library:D_SOD-323, F.Cu at (405.4, 94.9)
- added D25: ESD9B5.0ST5G, Diode_SMD:D_0402_1005Metric, F.Cu at (393.7, 79.6)
- added D26: 1N5819WS, A_HDJ_Library:D_SOD-323, F.Cu at (411.7, 150.1)
- added D27: 1N5819WS, A_HDJ_Library:D_SOD-323, F.Cu at (411.7, 153.0)
- added D3: ESD5V0B03, A_HDJ_Library:D_0402_1005Metric, F.Cu at (384.1, 139.6)
- added D4: 1N5819WS, A_HDJ_Library:D_SOD-323, F.Cu at (371.1, 154.2)
- added D5: ESD5V0B03, A_HDJ_Library:D_0402_1005Metric, F.Cu at (328.1, 126.3)
- added D6: ESD5V0B03, A_HDJ_Library:D_0402_1005Metric, F.Cu at (328.1, 128.3)
- added D7: ESD5V0B03, A_HDJ_Library:D_0402_1005Metric, F.Cu at (328.1, 130.3)
- added D8: ESD5V0B03, A_HDJ_Library:D_0402_1005Metric, F.Cu at (328.1, 132.3)
- added D9: LED_G, A_HDJ_Library:LED_0603_1608Metric, F.Cu at (346.6, 132.9)
- added F1: 6V/50mA, A_HDJ_Library:R_0603_1608Metric, F.Cu at (375.2, 154.0)
- added F2: 6V/1A, A_HDJ_Library:Fuse_0805_2012Metric, F.Cu at (324.4, 126.8)
- added F3: 6V/1A, A_HDJ_Library:Fuse_0805_2012Metric, F.Cu at (324.4, 129.8)
- added F4: 6V/1A, A_HDJ_Library:Fuse_0805_2012Metric, F.Cu at (324.4, 132.7)
- added F5: 6V/1A, A_HDJ_Library:Fuse_0805_2012Metric, F.Cu at (324.4, 135.7)
- added J1: Conn_01x03_Pin, A_HDJ_Library:PinHeader_1x03_P2.54mm_Vertical, F.Cu at (305.8, 97.3)
- added J10: Conn_01x03_Pin, A_HDJ_Library:PinHeader_1x03_P2.54mm_Vertical, F.Cu at (370.0, 121.2)
- added J11: Conn_01x03_Pin, A_HDJ_Library:PinHeader_1x03_P2.54mm_Vertical, F.Cu at (374.7, 121.2)
- added J12: Conn_01x04_Pin, A_HDJ_Library:PinHeader_1x04_P2.54mm_Vertical, F.Cu at (374.7, 109.0)
- added J13: Conn_01x04_Pin, A_HDJ_Library:PinHeader_1x04_P2.54mm_Vertical, F.Cu at (379.3, 109.0)
- added J14: Conn_01x03_Pin, A_HDJ_Library:PinHeader_1x03_P2.54mm_Vertical, F.Cu at (379.3, 121.2)
- added J15: Bus_M.2_Socket_M, A_HDJ_Library:PCIe_M.2_Connectors_P=0.5mm_H=4.2mm_KeyM, F.Cu at (348.5, 112.8)
- added J16: Bus_M.2_Socket_E, A_HDJ_Library:PCIe_M.2_Connectors_P=0.5mm_H=4.2mm_KeyE, F.Cu at (339.2, 121.5)
- added J17: Barrel_Jack_Switch, A_HDJ_Library:DC_Jack_DC007B_30V_10A, F.Cu at (402.9, 74.7)
- added J19: Conn_01x04_Pin, A_HDJ_Library:PinHeader_1x04_P2.54mm_Vertical, F.Cu at (384.0, 109.0)
- added J2: Bus_PCI_Express_x4, A_HDJ_Library:PCIe_x4_Gen3Slot_Connectors, F.Cu at (387.6, 32.6)
- added J20: Conn_01x04_Pin, A_HDJ_Library:PinHeader_1x04_P2.54mm_Vertical, F.Cu at (388.6, 109.0)
- added J21: Conn_01x04_Pin, A_HDJ_Library:PinHeader_1x04_P2.54mm_Vertical, F.Cu at (393.3, 109.0)
- added J3: HDMI_A, A_HDJ_Library:HDMI_A_Molex_208658-1001_Horizontal, F.Cu at (368.7, 143.7)
- added J4: USB3_A_Stacked, A_HDJ_Library:USB3_A_Molex_48406-0001_Horizontal_Stacked, F.Cu at (309.3, 132.4)
- added J5: USB_A_Stacked, A_HDJ_Library:USB_A_CUI_UJ2-ADH-TH_Horizontal_Stacked, F.Cu at (317.5, 112.5)
- added J6: RJ45_RB1-125B8G1A, A_HDJ_Library:RJ45_UDE_RB1-125B8G1A, F.Cu at (401.9, 109.7)
- added J7: Conn_01x04_Pin, A_HDJ_Library:PinHeader_1x04_P2.54mm_Vertical, F.Cu at (365.4, 109.0)
- added J8: Conn_01x03_Pin, A_HDJ_Library:PinHeader_1x03_P2.54mm_Vertical, F.Cu at (365.4, 121.2)
- added J9: Conn_01x04_Pin, A_HDJ_Library:PinHeader_1x04_P2.54mm_Vertical, F.Cu at (370.0, 109.0)
- added L1: 2.2uH/4.3A, A_HDJ_Library:L_Sunlord_SWPA4020S, F.Cu at (386.8, 89.0)
- added L2: 2.2uH/4.3A, A_HDJ_Library:L_Sunlord_SWPA4020S, F.Cu at (386.8, 94.6)
- added M1: Fan_4pin, A_HDJ_Library:JST_PH_B4B-PH-K_1x04_P2.00mm_Vertical, F.Cu at (400.6, 139.4)
- added M2: Fan_4pin, A_HDJ_Library:JST_PH_B4B-PH-K_1x04_P2.00mm_Vertical, F.Cu at (400.6, 145.9)
- added Q1: 2SK3018, A_HDJ_Library:SOT-23, F.Cu at (380.2, 136.9)
- added Q2: 2SK3018, A_HDJ_Library:SOT-23, F.Cu at (380.2, 141.3)
- added Q3: 2SK3018, A_HDJ_Library:SOT-23, F.Cu at (380.2, 145.8)
- added Q4: 2SK3018, A_HDJ_Library:SOT-23, F.Cu at (380.2, 150.2)
- added Q5: 2N7002, A_HDJ_Library:SOT-23, F.Cu at (394.5, 61.1)
- added Q6: 2N7002, A_HDJ_Library:SOT-23, F.Cu at (394.5, 65.5)
- added Q7: AON7262E, A_HDJ_Library:MOSFET_PDFN8_3.3x3.3, F.Cu at (400.1, 91.5)
- added Q8: 2N7002, A_HDJ_Library:SOT-23, F.Cu at (394.5, 70.0)
- added R10: 470R/1%, A_HDJ_Library:R_0402_1005Metric, F.Cu at (387.0, 141.6)
- added R11: 1k/1%, A_HDJ_Library:R_0402_1005Metric, F.Cu at (387.0, 143.6)
- added R13: 470R/1%, A_HDJ_Library:R_0402_1005Metric, F.Cu at (387.0, 145.6)
- added R14: 470R/1%, A_HDJ_Library:R_0402_1005Metric, F.Cu at (387.0, 147.6)
- added R15: 2.2k/1%, A_HDJ_Library:R_0402_1005Metric, F.Cu at (389.9, 135.6)
- added R16: 470R/1%, A_HDJ_Library:R_0402_1005Metric, F.Cu at (389.9, 137.6)
- added R17: 470R/1%, A_HDJ_Library:R_0402_1005Metric, F.Cu at (389.9, 139.6)
- added R18: 2.2k/1%, A_HDJ_Library:R_0402_1005Metric, F.Cu at (389.9, 141.6)
- added R19: 2.2k/1%, A_HDJ_Library:R_0402_1005Metric, F.Cu at (389.9, 143.6)
- added R20: 10k/1%, A_HDJ_Library:R_0402_1005Metric, F.Cu at (419.2, 119.5)
- added R21: 10k/1%, A_HDJ_Library:R_0402_1005Metric, F.Cu at (419.2, 121.5)
- added R22: 2.49k/1%, A_HDJ_Library:R_0603_1608Metric, F.Cu at (422.6, 119.7)
- added R23: 1M/1%, A_HDJ_Library:R_0402_1005Metric, F.Cu at (419.2, 123.4)
- added R24: 470R/1%, A_HDJ_Library:R_0402_1005Metric, F.Cu at (419.2, 125.4)
- added R25: 470R/1%, A_HDJ_Library:R_0402_1005Metric, F.Cu at (419.2, 127.4)
- added R27: 0R/1%, A_HDJ_Library:R_0402_1005Metric, F.Cu at (334.5, 107.6)
- added R29: 0R/1%, A_HDJ_Library:R_0402_1005Metric, F.Cu at (334.5, 109.6)
- added R3: 2.2k/1%, A_HDJ_Library:R_0402_1005Metric, F.Cu at (384.1, 141.6)
- added R30: 2.2K/1%, A_HDJ_Library:R_0402_1005Metric, F.Cu at (334.5, 111.6)
- added R32: 0R/1%, A_HDJ_Library:R_0402_1005Metric, F.Cu at (334.5, 113.6)
- added R33: 0R/1%, A_HDJ_Library:R_0402_1005Metric, F.Cu at (334.5, 115.6)
- added R34: 10k/1%, A_HDJ_Library:R_0402_1005Metric, F.Cu at (334.5, 117.6)
- added R35: 10k/1%, A_HDJ_Library:R_0402_1005Metric, F.Cu at (334.5, 119.6)
- added R36: 10k/1%, A_HDJ_Library:R_0402_1005Metric, F.Cu at (410.4, 69.8)
- added R37: 1k/1%, A_HDJ_Library:R_0402_1005Metric, F.Cu at (413.3, 59.8)
- added R38: 10k/1%, A_HDJ_Library:R_0402_1005Metric, F.Cu at (413.3, 61.8)
- added R39: 2.2k/1%, A_HDJ_Library:R_0402_1005Metric, F.Cu at (413.3, 63.8)
- added R4: 1M/1%, A_HDJ_Library:R_0402_1005Metric, F.Cu at (384.1, 143.6)
- added R40: 10k/1%, A_HDJ_Library:R_0402_1005Metric, F.Cu at (413.3, 65.8)
- added R41: 21.5k/1%, A_HDJ_Library:R_0402_1005Metric, F.Cu at (413.3, 67.8)
- added R42: 21.5k/1%, A_HDJ_Library:R_0402_1005Metric, F.Cu at (413.3, 69.8)
- added R43: 56k/1%, A_HDJ_Library:R_0402_1005Metric, F.Cu at (416.2, 59.8)
- added R44: 100k/1%, A_HDJ_Library:R_0402_1005Metric, F.Cu at (416.2, 61.8)
- added R45: 100k/1%, A_HDJ_Library:R_0402_1005Metric, F.Cu at (416.2, 63.8)
- added R46: 100k/1%, A_HDJ_Library:R_0402_1005Metric, F.Cu at (416.2, 65.8)
- added R47: 1k/1%, A_HDJ_Library:R_0402_1005Metric, F.Cu at (416.2, 67.8)
- added R48: 100R/1%, A_HDJ_Library:R_0402_1005Metric, F.Cu at (416.2, 69.8)
- added R49: 10k/1%, A_HDJ_Library:R_0402_1005Metric, F.Cu at (419.1, 59.8)
- added R5: 2.2k/1%, A_HDJ_Library:R_0402_1005Metric, F.Cu at (384.1, 145.6)
- added R50: 10k/1%, A_HDJ_Library:R_0402_1005Metric, F.Cu at (419.1, 61.8)
- added R51: 100k/1%, A_HDJ_Library:R_0402_1005Metric, F.Cu at (419.1, 63.8)
- added R52: 2.2k/1%, A_HDJ_Library:R_0402_1005Metric, F.Cu at (419.1, 65.8)
- added R53: 2.2k/1%, A_HDJ_Library:R_0402_1005Metric, F.Cu at (419.1, 67.8)
- added R54: 21.5k/1%, A_HDJ_Library:R_0402_1005Metric, F.Cu at (419.1, 69.8)
- added R55: 100R/1%, A_HDJ_Library:R_0402_1005Metric, F.Cu at (422.1, 59.8)
- added R56: 10k/1%, A_HDJ_Library:R_0402_1005Metric, F.Cu at (422.1, 61.8)
- added R57: 75k/1%, A_HDJ_Library:R_0402_1005Metric, F.Cu at (422.1, 63.8)
- added R58: 10k/1%, A_HDJ_Library:R_0402_1005Metric, F.Cu at (422.1, 65.8)
- added R59: 21.5k/1%, A_HDJ_Library:R_0402_1005Metric, F.Cu at (422.1, 67.8)
- added R6: 21.5k/1%, A_HDJ_Library:R_0402_1005Metric, F.Cu at (384.1, 147.6)
- added R60: 4.7k/1%, A_HDJ_Library:R_0402_1005Metric, F.Cu at (422.1, 69.8)
- added R63: 10k/1%, A_HDJ_Library:R_0402_1005Metric, F.Cu at (411.0, 137.7)
- added R64: 4.7k/1%, A_HDJ_Library:R_0402_1005Metric, F.Cu at (411.0, 139.7)
- added R65: 4.7k/1%, A_HDJ_Library:R_0402_1005Metric, F.Cu at (411.0, 141.6)
- added R66: 21.5k/1%, A_HDJ_Library:R_0402_1005Metric, F.Cu at (411.0, 143.6)
- added R67: 21.5k/1%, A_HDJ_Library:R_0402_1005Metric, F.Cu at (411.0, 145.6)
- added R68: 21.5k/1%, A_HDJ_Library:R_0402_1005Metric, F.Cu at (411.0, 147.6)
- added R69: 100R/1%, A_HDJ_Library:R_0402_1005Metric, F.Cu at (413.9, 137.7)
- added R7: 470R/1%, A_HDJ_Library:R_0402_1005Metric, F.Cu at (387.0, 135.6)
- added R70: 21.5k/1%, A_HDJ_Library:R_0402_1005Metric, F.Cu at (413.9, 139.7)
- added R71: 100R/1%, A_HDJ_Library:R_0402_1005Metric, F.Cu at (413.9, 141.6)
- added R72: 4.7k/1%, A_HDJ_Library:R_0402_1005Metric, F.Cu at (413.9, 143.6)
- added R74: 4.7k/1%, A_HDJ_Library:R_0402_1005Metric, F.Cu at (413.9, 145.6)
- added R8: 470R/1%, A_HDJ_Library:R_0402_1005Metric, F.Cu at (387.0, 137.6)
- added R9: 470R/1%, A_HDJ_Library:R_0402_1005Metric, F.Cu at (387.0, 139.6)
- added SW1: SW_Push, A_HDJ_Library:SW_Push_6x6x6, F.Cu at (414.4, 77.5)
- added SW2: SW_Push, A_HDJ_Library:SW_Push_6x6x6, F.Cu at (414.4, 84.6)
- added U1: D3V3XA4B10LP, A_HDJ_Library:Diodes_UDFN-10_1.0x2.5mm_P0.5mm, F.Cu at (364.5, 154.7)
- added U10: ULC0524P, A_HDJ_Library:Diodes_UDFN-10_1.0x2.5mm_P0.5mm, F.Cu at (367.5, 130.6)
- added U11: ULC0524P, A_HDJ_Library:Diodes_UDFN-10_1.0x2.5mm_P0.5mm, F.Cu at (370.4, 130.6)
- added U12: ULC0524P, A_HDJ_Library:Diodes_UDFN-10_1.0x2.5mm_P0.5mm, F.Cu at (373.4, 130.6)
- added U13: TL431DBZ, A_HDJ_Library:SOT-23, F.Cu at (394.5, 74.4)
- added U14: USB PD等快充协议受电芯片-CH224K-ESSOP10, A_HDJ_Library:ESSOP-10-1EP_3.9x5mm_P1.0mm_EP3.2x2.3, F.Cu at (418.0, 91.6)
- added U15: LM2734X, A_HDJ_Library:TSOT-23-6, F.Cu at (411.5, 90.4)
- added U16: LM2734X, A_HDJ_Library:TSOT-23-6, F.Cu at (411.5, 95.0)
- added U17: ULC0524P, A_HDJ_Library:Diodes_UDFN-10_1.0x2.5mm_P0.5mm, F.Cu at (376.3, 130.6)
- added U2: D3V3XA4B10LP, A_HDJ_Library:Diodes_UDFN-10_1.0x2.5mm_P0.5mm, F.Cu at (367.5, 154.7)
- added U3: D3V3XA4B10LP, A_HDJ_Library:Diodes_UDFN-10_1.0x2.5mm_P0.5mm, F.Cu at (323.7, 139.2)
- added U4: D3V3XA4B10LP, A_HDJ_Library:Diodes_UDFN-10_1.0x2.5mm_P0.5mm, F.Cu at (326.6, 139.2)
- added U5: D3V3XA4B10LP, A_HDJ_Library:Diodes_UDFN-10_1.0x2.5mm_P0.5mm, F.Cu at (329.6, 139.2)
- added U6: RTL8111H-CG-RH, A_HDJ_Library:QFN-32-1EP_4x4mm_P0.4mm_EP2.65x2.65mm, F.Cu at (420.8, 131.5)
- added U9: ULC0524P, A_HDJ_Library:Diodes_UDFN-10_1.0x2.5mm_P0.5mm, F.Cu at (364.5, 130.6)
Other:
- board outline added: 164.2 x 98.5 mm

Commit message: fix: Set missing footprints and fixed missing pin-pad connections.
- J15, J16 missing MP1 and MP2 pins. Fixed in pin table within the symbol editor for each symbol.
- A ll USB receptacles J4, J5, J18 had mismatched pin numbers for the pcb symbol footprint. Renamed to match.
- Fixed various DNP components that were not excluded from the board.
- Fixed remaining missing footprints.
Parts:
- added BT1: Battery_Cell, A_HDJ_Library:Battery_Holder_CR1220_S8411-45R, F.Cu at (315.5, 99.9)
- added FID78: Fiducial, A_HDJ_Library:Fiducial_0.5mm_Mask1mm, F.Cu at (431.4, 94.3)
- added FID79: Fiducial, A_HDJ_Library:Fiducial_0.5mm_Mask1mm, F.Cu at (431.4, 96.9)
- added H1: MountingHole_Pad, A_HDJ_Library:MountingHole_3.2mm_M3_Pad_Via, F.Cu at (426.2, 97.0)
- added H2: MountingHole_Pad, A_HDJ_Library:MountingHole_3.2mm_M3_Pad_Via, F.Cu at (426.2, 105.0)
- added H3: MountingHole_Pad, A_HDJ_Library:MountingHole_3.2mm_M3_Pad_Via, F.Cu at (426.2, 112.9)
- added H4: MountingHole_Pad, A_HDJ_Library:MountingHole_3.2mm_M3_Pad_Via, F.Cu at (426.2, 120.9)
- added H5: MountingHole_Pad, A_HDJ_Library:MountingHole_3mm_M2_Pad_TopOnly, F.Cu at (327.1, 92.5)
- added H6: MountingHole_Pad, A_HDJ_Library:MountingHole_3mm_M2_Pad_TopOnly, F.Cu at (327.1, 99.7)
- added H7: MountingHole_M2.0, A_HDJ_Library:MountingHole_2.7mm_M2_Pad_TopOnly, F.Cu at (391.5, 96.6)
- added H8: MountingHole_M2.0, A_HDJ_Library:MountingHole_2.7mm_M2_Pad_TopOnly, F.Cu at (391.5, 103.8)
- added J18: USB_C_Receptacle_USB2.0_16P, A_HDJ_Library:USB_C_Receptacle_G-Switch_GT-USB-7010ASV, F.Cu at (338.3, 133.3)
- added JP1: Jumper_3_Bridged12, A_HDJ_Library:PinHeader_1x03_P2.54mm_Vertical, F.Cu at (329.9, 148.0)
- added R1: 1k/1%, A_HDJ_Library:R_0402_1005Metric, F.Cu at (332.1, 89.9)
- added R2: 10k/1%, A_HDJ_Library:R_0402_1005Metric, F.Cu at (332.1, 91.9)
- added R76: 100k/1%, A_HDJ_Library:R_0402_1005Metric, F.Cu at (332.1, 93.9)
- added R77: 100k/1%, A_HDJ_Library:R_0402_1005Metric, F.Cu at (332.1, 95.9)
- added R78: 10k/1%, A_HDJ_Library:R_0402_1005Metric, F.Cu at (332.1, 97.9)
- added R79: 10k/1%, A_HDJ_Library:R_0402_1005Metric, F.Cu at (332.1, 99.9)
- added TP10: TestPoint, A_HDJ_Library:TestPoint_Pad_D1.5mm, F.Cu at (344.9, 139.8)
- added TP11: TestPoint, A_HDJ_Library:TestPoint_Pad_D1.5mm, F.Cu at (436.2, 141.6)
- added TP12: TestPoint, A_HDJ_Library:TestPoint_Pad_D1.5mm, F.Cu at (436.2, 145.1)
- added TP13: TestPoint, A_HDJ_Library:TestPoint_Pad_D1.5mm, F.Cu at (344.9, 143.3)
- added TP2: TestPoint, A_HDJ_Library:TestPoint_Pad_D1.5mm, F.Cu at (405.5, 119.8)
- added TP3: TestPoint, A_HDJ_Library:TestPoint_Pad_D1.5mm, F.Cu at (334.3, 139.8)
- added TP4: TestPoint, A_HDJ_Library:TestPoint_Pad_D1.5mm, F.Cu at (334.3, 143.3)
- added TP5: TestPoint, A_HDJ_Library:TestPoint_Pad_D1.5mm, F.Cu at (337.8, 139.8)
- added TP6: TestPoint, A_HDJ_Library:TestPoint_Pad_D1.5mm, F.Cu at (337.8, 143.3)
- added TP78: TestPoint, A_HDJ_Library:TestPoint_Pad_D1.5mm, F.Cu at (335.3, 100.4)
- added TP8: TestPoint, A_HDJ_Library:TestPoint_Pad_D1.5mm, F.Cu at (341.4, 139.8)
- added TP9: TestPoint, A_HDJ_Library:TestPoint_Pad_D1.5mm, F.Cu at (341.4, 143.3)
- added U7: ULC0524P, A_HDJ_Library:Diodes_UDFN-10_1.0x2.5mm_P0.5mm, F.Cu at (0.97, 1.52)
- added U8: ULC0524P, A_HDJ_Library:Diodes_UDFN-10_1.0x2.5mm_P0.5mm, F.Cu at (3.92, 1.52)
- added Y1: 25MHz, A_HDJ_Library:Crystal_SMD_3225-4Pin_3.2x2.5mm, F.Cu at (375.9, 126.9)
- moved SW1 115.7 mm to (321.1, 145.8)
- moved SW2 115.7 mm to (321.1, 152.9)
- moved U15 114.0 mm to (310.1, 142.5)
- moved U16 114.0 mm to (310.1, 147.0)
- moved Q7 108.2 mm to (310.7, 152.4)
- moved C26 100.1 mm to (409.2, 53.8)
- moved C27 100.1 mm to (409.2, 55.8)
- moved C28 100.1 mm to (409.2, 57.8)
- moved C29 100.1 mm to (409.2, 59.7)
- moved C30 100.1 mm to (412.6, 54.1)
- moved C31 100.1 mm to (412.6, 56.6)
- moved C32 100.1 mm to (412.6, 59.1)
- moved F2 100.1 mm to (408.8, 73.0)
- moved F3 100.1 mm to (408.8, 76.0)
- moved F4 100.1 mm to (408.8, 78.9)
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Connections:
- J15 pad MP1: (no net) -> GND
- J15 pad MP2: (no net) -> GND
- J16 pad MP1: (no net) -> GND
- J16 pad MP2: (no net) -> GND
- J4 pad 19: (no net) -> GND
- J5 pad 9: (no net) -> GND

Commit message: fix: Fixed DNP parts populating on the board.
Parts:
- removed C1, C2, C3, C4, C5, C6, C7, C8: 220nF/50V, A_HDJ_Library:C_0402_1005Metric
- removed C10, C13, C15, C85, C9: 100nF/50V, A_HDJ_Library:C_0402_1005Metric
- removed C11: 100uF/25V, A_HDJ_Library:CP_Elec_6.3x7.7
- removed C14: 10uF/10V, A_HDJ_Library:C_0402_1005Metric
- removed C16: 560uF/25V, A_HDJ_Library:CP_Elec_6.3x7.7
- removed C62, C63: 1uF/16V, A_HDJ_Library:C_0402_1005Metric
- removed D23: LED, A_HDJ_Library:LED_0603_1608Metric
- removed D27: 1N5819WS, A_HDJ_Library:D_SOD-323
- removed J2: Bus_PCI_Express_x4, A_HDJ_Library:PCIe_x4_Gen3Slot_Connectors
- removed M2: Fan_4pin, A_HDJ_Library:JST_PH_B4B-PH-K_1x04_P2.00mm_Vertical
- removed Q5, Q6: 2N7002, A_HDJ_Library:SOT-23
- removed Q7: AON7262E, A_HDJ_Library:MOSFET_PDFN8_3.3x3.3
- removed R38, R40, R50, R56, R63: 10k/1%, A_HDJ_Library:R_0402_1005Metric
- removed R39: 2.2k/1%, A_HDJ_Library:R_0402_1005Metric
- removed R41, R42, R54, R66, R67, R70: 21.5k/1%, A_HDJ_Library:R_0402_1005Metric
- removed R44, R45: 100k/1%, A_HDJ_Library:R_0402_1005Metric
- removed R64, R65, R74: 4.7k/1%, A_HDJ_Library:R_0402_1005Metric
- removed R71: 100R/1%, A_HDJ_Library:R_0402_1005Metric
- removed TP8, TP9: TestPoint, A_HDJ_Library:TestPoint_Pad_D1.5mm
- removed U13: TL431DBZ, A_HDJ_Library:SOT-23
- removed U7, U8: ULC0524P, A_HDJ_Library:Diodes_UDFN-10_1.0x2.5mm_P0.5mm
- moved A1 42.0 mm to (339.0, 69.5), turned to 180 degrees

Commit message: feat(layout): Main component placement.
Parts:
- moved H2 357.7 mm to (71.0, 62.5)
- moved H3 357.3 mm to (71.0, 152.0)
- moved J21 343.7 mm to (81.8, 59.9)
- moved J20 335.2 mm to (85.8, 59.9)
- moved J13 334.0 mm to (77.8, 59.9)
- moved J19 322.4 mm to (94.2, 59.9)
- moved J14 321.3 mm to (83.0, 149.0)
- moved J11 320.6 mm to (79.0, 149.0)
- moved J12 317.7 mm to (89.8, 59.9)
- moved H7 316.5 mm to (75.2, 109.5)
- moved J9 304.4 mm to (98.8, 59.9)
- moved J10 303.2 mm to (91.8, 149.0)
- moved J8 302.6 mm to (87.8, 149.0)
- moved J7 296.0 mm to (102.8, 59.9)
- moved J16 289.5 mm to (109.0, 100.2), turned to -90 degrees
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Other:
- board size 164.2 x 98.5 mm -> 462.5 x 294.6 mm

Commit message: feat(layout): Respositioned M.2 keys for better routing.
- Repositioned other components that interfered.
Parts:
- moved C56 293.1 mm to (108.7, 87.9), turned to 180 degrees
- moved C55 292.9 mm to (108.7, 86.9), turned to 180 degrees
- moved C50 287.8 mm to (108.8, 115.6), turned to 180 degrees
- moved C49 287.8 mm to (108.8, 116.6), turned to 180 degrees
- moved H8 147.3 mm to (72.0, 113.5), turned to 180 degrees
- moved J6 118.0 mm to (191.0, 136.9), turned to 0 degrees
- moved J15 93.1 mm to (102.0, 113.5), turned to -90 degrees
- moved SW1 59.0 mm to (226.2, 104.2), turned to -90 degrees
- moved SW2 39.7 mm to (226.2, 118.2), turned to -90 degrees
- moved H7 21.7 mm to (72.0, 88.1)
- moved J16 21.7 mm to (105.8, 78.8)
- moved BT1 8.34 mm to (76.8, 138.2)
- moved A1 1.50 mm to (148.5, 118.4)

Commit message: feat(routing): Routed M.2 differential pairs and tuned skew for differential pairs.
Parts:
- moved C55 0.17 mm to (108.7, 87.0)
- moved C56 0.17 mm to (108.7, 88.0)
- moved C49 0.10 mm to (108.8, 116.5)
- moved C50 0.10 mm to (108.8, 115.5)
Routing:
- net /LattePanda Module/USB_2_P7-: track 0.00 -> 66.9 mm, vias 0 -> 2
- net /LattePanda Module/USB_2_P7+: track 0.00 -> 66.9 mm, vias 0 -> 2
- net /LattePanda Module/REFCLK_3-: track 0.00 -> 58.3 mm, vias 0 -> 2
- net /LattePanda Module/REFCLK_3+: track 0.00 -> 58.3 mm, vias 0 -> 2
- net /LattePanda Module/HSIO_3_TX-: track 0.00 -> 48.8 mm, vias 0 -> 2
- net /LattePanda Module/HSIO_3_TX+: track 0.00 -> 48.8 mm, vias 0 -> 2
- net /LattePanda Module/HSIO_3_RX-: track 0.00 -> 44.4 mm, vias 0 -> 2
- net /LattePanda Module/HSIO_3_RX+: track 0.00 -> 44.4 mm, vias 0 -> 2
- net /LattePanda Module/REFCLK_0+: track 0.00 -> 35.7 mm, vias 0 -> 2
- net /LattePanda Module/REFCLK_0-: track 0.00 -> 35.7 mm, vias 0 -> 2
- net /LattePanda Module/HSIO_2_RX+: track 0.00 -> 20.7 mm
- net /LattePanda Module/HSIO_2_RX-: track 0.00 -> 20.7 mm
- net /LattePanda Module/HSIO_2_TX-: track 0.00 -> 17.1 mm
- net /LattePanda Module/HSIO_2_TX+: track 0.00 -> 17.1 mm
- net /M.2 M Key/CON_PCIE_TX1-: track 0.00 -> 2.87 mm
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
Commit message: feat(routing): Routed low-speed M.2 signals to related resistors and components.
- Did not route signals directly to LattePandaMu, waiting until all differential pairs are routed.
- Did not route power.
Parts:
- moved TP2 335.3 mm to (70.2, 127.8)
- moved C60 312.8 mm to (92.8, 79.5), turned to -90 degrees
- moved C59 311.6 mm to (93.8, 79.5), turned to -90 degrees
- moved C58 310.3 mm to (94.8, 79.5), turned to -90 degrees
- moved C57 309.1 mm to (95.8, 79.5), turned to -90 degrees
- moved C54 305.1 mm to (94.8, 105.2), turned to -90 degrees
- moved C52 304.4 mm to (92.8, 105.2), turned to -90 degrees
- moved C53 304.0 mm to (95.8, 105.2), turned to -90 degrees
- moved C51 303.3 mm to (93.8, 105.2), turned to -90 degrees
- moved D9 301.1 mm to (108.8, 101.8), turned to 90 degrees
- moved R35 295.5 mm to (95.2, 91.8), turned to 180 degrees
- moved R33 295.3 mm to (95.2, 90.5), turned to 180 degrees
- moved R34 295.2 mm to (95.2, 93.0), turned to 180 degrees
- moved R29 294.3 mm to (95.2, 120.8), turned to 180 degrees
- moved R27 294.3 mm to (95.2, 117.0), turned to 180 degrees
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Routing:
- net Net-(J15-DEVSLP): track 0.00 -> 36.6 mm
- net Net-(D9-K): track 0.00 -> 13.6 mm
- net Net-(J16-SUSCLK): track 0.00 -> 2.77 mm
- net Net-(J16-~{W_DISABLE1}): track 0.00 -> 2.73 mm
- net Net-(J16-~{W_DISABLE2}): track 0.00 -> 2.66 mm
- net /M.2 M Key/~{CLKREQM}: track 0.00 -> 2.28 mm
- net +3.3V: track 0.00 -> 1.25 mm
Other:
- board size 462.5 x 294.6 mm -> 165 x 100 mm

Commit message: feat(routing): Routed hdmi differential pairs.
- TMDS_D1+/- shows + and - equal skew on both sides, so tuning was ignored for this pair.
Parts:
- moved R15 297.2 mm to (167.8, 162.8)
- moved C25 291.8 mm to (172.9, 179.0)
- moved D4 291.8 mm to (154.2, 179.7)
- moved F1 291.8 mm to (158.4, 179.5)
- moved Q2 291.8 mm to (163.3, 166.8)
- moved Q3 291.8 mm to (163.3, 171.3)
- moved R11 291.8 mm to (170.1, 169.1)
- moved R18 291.8 mm to (173.0, 167.1)
- moved R19 291.8 mm to (173.0, 169.1)
- moved R3 291.8 mm to (167.2, 167.1)
- moved R4 291.8 mm to (167.2, 169.1)
- moved R5 291.8 mm to (167.2, 171.1)
- moved R6 291.8 mm to (167.2, 173.1)
- moved Q1 291.7 mm to (163.3, 162.2)
- moved D1 291.3 mm to (166.8, 158.8), turned to 180 degrees
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Routing:
- net /HDMI/DDI_B_TX0-: track 0.00 -> 23.2 mm
- net /HDMI/DDI_B_TX0+: track 0.00 -> 23.2 mm
- net /HDMI/DDI_B_TX1+: track 0.00 -> 22.9 mm
- net /HDMI/DDI_B_TX1-: track 0.00 -> 22.9 mm
- net /HDMI/DDI_B_TX2-: track 0.00 -> 22.0 mm
- net /HDMI/DDI_B_TX2+: track 0.00 -> 22.0 mm
- net /HDMI/DDI_B_TX3-: track 0.00 -> 21.5 mm
- net /HDMI/DDI_B_TX3+: track 0.00 -> 21.5 mm
- net /HDMI/TMDS_D2-: track 0.00 -> 11.9 mm
- net /HDMI/TMDS_D2+: track 0.00 -> 11.9 mm
- net /HDMI/TMDS_CK-: track 0.00 -> 11.9 mm
- net /HDMI/TMDS_CK+: track 0.00 -> 11.9 mm
- net /HDMI/TMDS_D1+: track 0.00 -> 11.2 mm
- net /HDMI/TMDS_D1-: track 0.00 -> 11.2 mm
- net /HDMI/TMDS_D0-: track 0.00 -> 11.1 mm
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