File: ethernet.kicad_sch (KiCad schematic)
At the start: 0 parts

Commit message: feat(ethernet): Added Gigabit Ethernet implementation and connections.
Parts:
- added C33, C34, C35, C37, C38, C39, C40, C41, C42, C43, C45, C48: 100nF/50V, A_HDJ_Library:C_0402_1005Metric, symbol Device:C
- added C44: 10uF/50V, A_HDJ_Library:C_0402_1005Metric, symbol Device:C
- added C46, C47: 12pF/50V, A_HDJ_Library:C_0402_1005Metric, symbol Device:C
- added J6: RJ45_RB1-125B8G1A, A_HDJ_Library:RJ45_UDE_RB1-125B8G1A, symbol Connector:RJ45_RB1-125B8G1A
- added R20, R21: 10k/1%, A_HDJ_Library:R_0402_1005Metric, symbol Device:R
- added R22: 2.49k/1%, A_HDJ_Library:R_0603_1608Metric, symbol Device:R
- added R23: 1M/1%, A_HDJ_Library:R_0402_1005Metric, symbol Device:R
- added R24, R25: 470R/1%, A_HDJ_Library:R_0402_1005Metric, symbol Device:R
- added U6: RTL8111H-CG-RH, A_HDJ_Library:QFN-32-1EP_4x4mm_P0.4mm_EP2.65x2.65mm, symbol A_HDJ_Library:RTL8111H-CG-RH
- added U7, U8: ULC0524P, Package_DFN_QFN:Diodes_UDFN-10_1.0x2.5mm_P0.5mm, symbol Power_Protection:D3V3XA4B10LP
- added Y1: 25MHz, symbol Device:Crystal_GND24
Connections:
- new net: C43.2, U6.17 (HSOP)
- new net: R20.1, U6.20 (ISOLATEB)
- new net: C39.2, U6.18 (HSON)
- new net: C42.2, U6.13 (HSIP)
- new net: C46.1, R23.2, U6.29 (CKXTAL2), Y1.3
- new net: J6.L1, R25.1
- new net: C47.1, R23.1, U6.28 (CKXTAL1), Y1.1
- new net: J6.L3, R24.1
- new net: C48.2, J6.R1 (CT)
- new net: C38.2, U6.14 (HSIN)
- new net: R21.1, U6.21 (LANWAKEB)
- new net: R22.2, U6.31 (RSET)
- new net +1V0: C33.2, C34.2, C35.2, C40.2, C44.2, U6.22 (DVDD10), U6.24 (REGOUT), U6.3 (AVDD10), U6.30 (AVDD10), U6.8 (AVDD10)
- new net +3.3V: C37.2, C41.2, C45.2, R20.2, R21.2, R24.2, R25.2, U6.11 (AVDD33), U6.23 (VDDREG), U6.32 (AVDD33)
- new net GND: C33.1, C34.1, C35.1, C37.1, C40.1, C41.1, C44.1, C45.1, C46.2, C47.2, C48.1, J6.R10 (GND), J6.SH, R22.1, U6.33 (GND), U7.3 (VSS), U7.8 (VSS), U8.3 (VSS), U8.8 (VSS), Y1.2 (G), Y1.4 (G)
- new net GbE_PCIe_CLK+: U6.15 (REFCLK_P)
- new net GbE_PCIe_CLK-: U6.16 (REFCLK_N)
- new net GbE_PCIe_RX+: C43.1
- new net GbE_PCIe_RX-: C39.1
- new net GbE_PCIe_TX+: C42.1
- new net GbE_PCIe_TX-: C38.1
- new net LED0_100: U6.27 (LED0)
- new net LED1_1000: J6.L4, U6.26 (LED1)
- new net LED2_ACT: J6.L2, U6.25 (LED2)
- new net MDI0+: J6.R2 (TD1+), U6.1 (MDIP0), U8.5, U8.6 (NC)
- new net MDI0-: J6.R3 (TD1-), U6.2 (MDIN0), U8.4, U8.7 (NC)
- new net MDI1+: J6.R4 (TD2+), U6.4 (MDIP1), U8.2, U8.9 (NC)
- new net MDI1-: J6.R5 (TD2-), U6.5 (MDIN1), U8.1, U8.10 (NC)
- new net MDI2+: J6.R6 (TD3+), U6.6 (MDIP2), U7.5, U7.6 (NC)
- new net MDI2-: J6.R7 (TD3-), U6.7 (MDIN2), U7.4, U7.7 (NC)
- new net MDI3+: J6.R8 (TD4+), U6.9 (MDIP3), U7.2, U7.9 (NC)
- new net MDI3-: J6.R9 (TD4-), U6.10 (MDIN3), U7.1, U7.10 (NC)
- new net ~{PLT_RST}: U6.19 (PERSTB)
- no-connect marks 0 -> 2

Commit message: fix: Set missing footprints and fixed missing pin-pad connections.
- J15, J16 missing MP1 and MP2 pins. Fixed in pin table within the symbol editor for each symbol.
- A ll USB receptacles J4, J5, J18 had mismatched pin numbers for the pcb symbol footprint. Renamed to match.
- Fixed various DNP components that were not excluded from the board.
- Fixed remaining missing footprints.
Parts:
- U7, U8: footprint Package_DFN_QFN:Diodes_UDFN-10_1.0x2.5mm_P0.5mm -> A_HDJ_Library:Diodes_UDFN-10_1.0x2.5mm_P0.5mm
- Y1: footprint (none) -> A_HDJ_Library:Crystal_SMD_3225-4Pin_3.2x2.5mm

Commit message: feat(routing): Routed ethernet connections; still need to perform length tuning on differential pairs or rerouting.
Parts:
- U7, U8: now in the parts list
Connections:
- net MDI0+: now also U7.1, U7.10 (NC); no longer U8.5, U8.6 (NC)
- net MDI0-: now also U7.2, U7.9 (NC); no longer U8.4, U8.7 (NC)
- net MDI1+: now also U7.4, U7.7 (NC); no longer U8.2, U8.9 (NC)
- net MDI1-: now also U7.5, U7.6 (NC); no longer U8.1, U8.10 (NC)
- net MDI2+: now also U8.5, U8.6 (NC); no longer U7.5, U7.6 (NC)
- net MDI2-: now also U8.4, U8.7 (NC); no longer U7.4, U7.7 (NC)
- net MDI3+: now also U8.2, U8.9 (NC); no longer U7.2, U7.9 (NC)
- net MDI3-: now also U8.1, U8.10 (NC); no longer U7.1, U7.10 (NC)
- net HSO+: now reaches C43.2, U6.17 (HSOP)
- net HSO-: now reaches C39.2, U6.18 (HSON)
- net HSI+: now reaches C42.2, U6.13 (HSIP)
- net HSI-: now reaches C38.2, U6.14 (HSIN)
Changed lines of the file:
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@@
 		)
 	)
+	(label "MDI2-"
+		(at 203.2 30.48 0)
+		(effects
+			(font
+				(size 1.27 1.27)
+			)
+			(justify left bottom)
+		)
+	)
+	(label "MDI2+"
+		(at 203.2 35.56 0)
+		(effects
+			(font
+				(size 1.27 1.27)
+			)
+			(justify left bottom)
+		)
+	)
 	(label "MDI1-"
 		(at 160.02 90.17 0)
@@
 		)
 	)
-	(label "MDI0+"
-		(at 203.2 35.56 0)
+	(label "HSI-"
+		(at 110.49 110.49 0)
 		(effects
 			(font
@@
 		)
 	)
-	(label "MDI3-"
-		(at 127 30.48 180)
+	(label "HSO-"
+		(at 110.49 115.57 0)
 		(effects
 			(font
 				(size 1.27 1.27)
 			)
-			(justify right bottom)
+			(justify left bottom)
 		)
 	)
@@
 		)
 	)
-	(label "MDI3+"
-		(at 127 35.56 180)
+	(label "HSI+"
+		(at 110.49 113.03 0)
+		(effects
+			(font
+				(size 1.27 1.27)
+			)
+			(justify left bottom)
+		)
+	)
+	(label "MDI3-"
+		(at 177.8 30.48 180)
 		(effects
 			(font
@@
 		)
 	)
-	(label "MDI1+"
-		(at 177.8 35.56 180)
+	(label "HSO+"
+		(at 110.49 118.11 0)
 		(effects
 			(font
 				(size 1.27 1.27)
 			)
-			(justify right bottom)
+			(justify left bottom)
 		)
 	)
 	(label "MDI0-"
-		(at 203.2 30.48 0)
+		(at 127 35.56 180)
 		(effects
 			(font
 				(size 1.27 1.27)
 			)
-			(justify left bottom)
+			(justify right bottom)
 		)
 	)
 	(label "MDI3+"
-		(at 160.02 82.55 0)
+		(at 177.8 35.56 180)
+		(effects
+			(font
+				(size 1.27 1.27)
+			)
+			(justify right bottom)
+		)
+	)
+	(label "MDI1-"
+		(at 152.4 35.56 0)
 		(effects
 			(font
@@
 		)
 	)
-	(label "MDI0-"
-		(at 160.04 95.25 0)
+	(label "MDI3+"
+		(at 160.02 82.55 0)
 		(effects
 			(font
@@
 		)
 	)
-	(label "MDI1-"
-		(at 177.8 30.48 180)
+	(label "MDI0-"
+		(at 160.04 95.25 0)
 		(effects
 			(font
 				(size 1.27 1.27)
 			)
-			(justify right bottom)
+			(justify left bottom)
 		)
 	)
-	(label "MDI2-"
+	(label "MDI1+"
 		(at 152.4 30.48 0)
 		(effects
@@
 		)
 	)
-	(label "MDI2-"
-		(at 160.02 85.09 0)
+	(label "MDI0+"
+		(at 127 30.48 180)
 		(effects
 			(font
 				(size 1.27 1.27)
 			)
-			(justify left bottom)
+			(justify right bottom)
 		)
 	)
-	(label "MDI2+"
-		(at 152.4 35.56 0)
+	(label "MDI2-"
+		(at 160.02 85.09 0)
 		(effects
 			(font
@@
 		(body_style 1)
 		(exclude_from_sim no)
-		(in_bom no)
-		(on_board no)
+		(in_bom yes)
+		(on_board yes)
 		(in_pos_files yes)
 		(dnp yes)
@@
 		(body_style 1)
 		(exclude_from_sim no)
-		(in_bom no)
-		(on_board no)
+		(in_bom yes)
+		(on_board yes)
 		(in_pos_files yes)
 		(dnp yes)
