File: m2_em_key.kicad_sch (KiCad schematic)
At the start: 0 parts

Commit message: feat(m.2): Added m.2 E and M keys
Parts:
- added C49, C50, C55, C56: 220nF/50V, A_HDJ_Library:C_0402_1005Metric, symbol Device:C
- added C51, C52, C53, C54, C57, C58, C59, C60: 100nF/50V, A_HDJ_Library:C_0402_1005Metric, symbol Device:C
- added D9: LED_G, A_HDJ_Library:LED_0603_1608Metric, symbol Device:LED
- added H7, H8: MountingHole_M2.0, A_HDJ_Library:MountingHole_2.75mm_M2_4.4mm_Pad_TopOnly, symbol Mechanical:MountingHole_Pad
- added J15: Bus_M.2_Socket_M, A_HDJ_Library:PCIe_M.2_Connectors_P=0.5mm_H=4.2mm_KeyM, symbol Connector:Bus_M.2_Socket_M
- added J16: Bus_M.2_Socket_E, A_HDJ_Library:PCIe_M.2_Connectors_P=0.5mm_H=4.2mm_KeyE, symbol Connector:Bus_M.2_Socket_E
- added R27, R29, R32, R33: 0R/1%, A_HDJ_Library:R_0402_1005Metric, symbol Device:R
- added R28: 0R/1%, Resistor_SMD:R_0402_1005Metric, symbol Device:R
- added R30: 2.2K/1%, A_HDJ_Library:R_0402_1005Metric, symbol Device:R
- added R34, R35: 10k/1%, A_HDJ_Library:R_0402_1005Metric, symbol Device:R
- added TP2: TestPoint, symbol Connector:TestPoint
Connections:
- new net: D9.2 (A), R30.1
- new net: D9.1 (K), J15.10 (DAS/~{DSS}/~{LED1})
- new net: J15.38 (DEVSLP), TP2.1
- new net: J15.68 (SUSCLK), R29.1
- new net: J15.69 (PEDET), R28.1
- new net: J16.50 (SUSCLK), R33.1
- new net: J16.54 (~{W_DISABLE2}), R35.1
- new net: J16.56 (~{W_DISABLE1}), R34.1
- new net +3.3V: C51.1, C52.1, C53.1, C54.1, C57.1, C58.1, C59.1, C60.1, J15.12 (3.3V), J15.14 (3.3V), J15.16 (3.3V), J15.18 (3.3V), J15.2 (3.3V), J15.4 (3.3V), J15.70 (3.3V), J15.72 (3.3V), J15.74 (3.3V), J16.2 (3.3V), J16.4 (3.3V), J16.72 (3.3V), J16.74 (3.3V), R30.2, R34.2, R35.2
- new net CON_PCIE_TX1+: C49.2, J15.49 (PETp0/SATA-A+)
- new net CON_PCIE_TX1-: C50.2, J15.47 (PETn0/SATA-A-)
- new net CON_PCIE_TX_0+: C55.2, J16.35 (PETp0)
- new net CON_PCIE_TX_0-: C56.2, J16.37 (PETn0)
- new net GND: C51.2, C52.2, C53.2, C54.2, C57.2, C58.2, C59.2, C60.2, H7.1, H8.1, J15.1 (GND), J15.15 (GND), J15.21 (GND), J15.27 (GND), J15.3 (GND), J15.33 (GND), J15.39 (GND), J15.45 (GND), J15.51 (GND), J15.57 (GND), J15.71 (GND), J15.73 (GND), J15.75 (GND), J15.9 (GND), J16.1 (GND), J16.18 (GND), J16.33 (GND), J16.39 (GND), J16.45 (GND), J16.51 (GND), J16.57 (GND), J16.63 (GND), J16.69 (GND), J16.7 (GND), J16.75 (GND), R27.2, R28.2, R32.2
- new net PCIE_RX_0+: J16.41 (PERp0)
- new net PCIE_RX_0-: J16.43 (PERn0)
- new net PCIE_RX_1+: J15.43 (PERp0/SATA-B-)
- new net PCIE_RX_1-: J15.41 (PERn0/SATA-B+)
- new net PCIE_TX_0+: C55.1
- new net PCIE_TX_0-: C56.1
- new net PCIE_TX_1+: C49.1
- new net PCIE_TX_1-: C50.1
- new net REFCLKE+: J16.47 (REFCLKp0)
- new net REFCLKE-: J16.49 (REFCLKn0)
- new net REFCLKM+: J15.55 (REFCLKp)
- new net REFCLKM-: J15.53 (REFCLKn)
- new net SUSCLK: R29.2, R33.2
- new net USB_2_P7+: J16.3 (USB_D+)
- new net USB_2_P7-: J16.5 (USB_D-)
- new net ~{CLKREQE}: J16.53 (~{CLKREQ0}), R32.1
- new net ~{CLKREQM}: J15.52 (~{CLKREQ}), R27.1
- new net ~{PLT_RST}: J15.50 (~{PERST}), J16.52 (~{PERST0})
- new net ~{WAKE}: J15.54 (~{PEWAKE}), J16.55 (~{PEWAKE0})
- no-connect marks 0 -> 50
Other:
- note added: "32.768kHz clock for low power mode"
- note added: "SSD active LED"

Commit message: fix: Set missing footprints and fixed missing pin-pad connections.
- J15, J16 missing MP1 and MP2 pins. Fixed in pin table within the symbol editor for each symbol.
- A ll USB receptacles J4, J5, J18 had mismatched pin numbers for the pcb symbol footprint. Renamed to match.
- Fixed various DNP components that were not excluded from the board.
- Fixed remaining missing footprints.
Parts:
- H7, H8: footprint A_HDJ_Library:MountingHole_2.75mm_M2_4.4mm_Pad_TopOnly -> A_HDJ_Library:MountingHole_2.7mm_M2_Pad_TopOnly; now left out of the parts list
- TP2: footprint (none) -> A_HDJ_Library:TestPoint_Pad_D1.5mm
Connections:
- net GND: now also J15.MP1, J15.MP2, J16.MP1, J16.MP2

Commit message: feat: Routed remaining m.2 passives and power.
- Fixed capacitor values.
Parts:
- C51, C53, C57, C59: value 100nF/50V -> 10uF/10V
Changed lines of the file:
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@@
 			)
 		)
-		(property "Value" "100nF/50V"
+		(property "Value" "10uF/10V"
 			(at 135.128 86.614 90)
 			(show_name no)
@@
 			)
 		)
-		(property "Value" "100nF/50V"
+		(property "Value" "10uF/10V"
 			(at 351.028 99.314 90)
 			(show_name no)
@@
 			)
 		)
-		(property "Value" "100nF/50V"
+		(property "Value" "10uF/10V"
 			(at 351.028 86.614 90)
 			(show_name no)
@@
 			)
 		)
-		(property "Value" "100nF/50V"
+		(property "Value" "10uF/10V"
 			(at 135.128 99.314 90)
 			(show_name no)
