File: gpio.kicad_sch (KiCad schematic)
At the start: 0 parts

Commit message: feat(gpio): Added gpio circuit and connections
Parts:
- added J10, J11, J14, J8: Conn_01x03_Pin, A_HDJ_Library:PinHeader_1x03_P2.54mm_Vertical, symbol Connector:Conn_01x03_Pin
- added J12, J13, J19, J20, J21, J7, J9: Conn_01x04_Pin, A_HDJ_Library:PinHeader_1x04_P2.54mm_Vertical, symbol Connector:Conn_01x04_Pin
- added U10, U11, U12, U17, U9: ULC0524P, A_HDJ_Library:Diodes_UDFN-10_1.0x2.5mm_P0.5mm, symbol Power_Protection:D3V3XA4B10LP
Connections:
- new net: U10.5, U10.6 (NC)
- new net: U12.5, U12.6 (NC)
- new net +3.3V: J13.1 (Pin_1), J13.2 (Pin_2), J13.3 (Pin_3), J13.4 (Pin_4), J14.1 (Pin_1), J14.2 (Pin_2), J14.3 (Pin_3), J21.1 (Pin_1), J21.2 (Pin_2), J21.3 (Pin_3), J21.4 (Pin_4)
- new net GND: J11.1 (Pin_1), J11.2 (Pin_2), J11.3 (Pin_3), J12.1 (Pin_1), J12.2 (Pin_2), J12.3 (Pin_3), J12.4 (Pin_4), J20.1 (Pin_1), J20.2 (Pin_2), J20.3 (Pin_3), J20.4 (Pin_4), U10.3 (VSS), U10.8 (VSS), U11.3 (VSS), U11.8 (VSS), U12.3 (VSS), U12.8 (VSS), U17.3 (VSS), U17.8 (VSS), U9.3 (VSS), U9.8 (VSS)
- new net GPP_D0: J19.1 (Pin_1), U17.1, U17.10 (NC)
- new net GPP_D1: J19.2 (Pin_2), U17.2, U17.9 (NC)
- new net GPP_D2: J19.3 (Pin_3), U17.4, U17.7 (NC)
- new net GPP_D3: J19.4 (Pin_4), U17.5, U17.6 (NC)
- new net I2C2_SCL: J9.1 (Pin_1), U11.1, U11.10 (NC)
- new net I2C2_SDA: J7.1 (Pin_1), U9.1, U9.10 (NC)
- new net I2C3_SCL: J9.2 (Pin_2), U11.2, U11.9 (NC)
- new net I2C3_SDA: J7.2 (Pin_2), U9.2, U9.9 (NC)
- new net I2C4_SCL: J9.3 (Pin_3), U11.4, U11.7 (NC)
- new net I2C4_SDA: J7.3 (Pin_3), U9.4, U9.7 (NC)
- new net I2C5_SCL: J9.4 (Pin_4), U11.5, U11.6 (NC)
- new net I2C5_SDA: J7.4 (Pin_4), U9.5, U9.6 (NC)
- new net SOC_UART0_RX: J8.1 (Pin_1), U10.1, U10.10 (NC)
- new net SOC_UART0_TX: J10.1 (Pin_1), U12.1, U12.10 (NC)
- new net SOC_UART1_RX: J8.2 (Pin_2), U10.2, U10.9 (NC)
- new net SOC_UART1_TX: J10.2 (Pin_2), U12.2, U12.9 (NC)
- new net SOC_UART2_RX: J8.3 (Pin_3), U10.4, U10.7 (NC)
- new net SOC_UART2_TX: J10.3 (Pin_3), U12.4, U12.7 (NC)
Other:
- note added: "GPIO"
- note added: "I2C"
- note added: "UART"
- title: (none) -> GPIO

Commit message: feat(routing): GPIO routing
Connections:
- net I2C2_SCL: now also U9.2, U9.9 (NC); no longer U11.1, U11.10 (NC)
- net I2C3_SCL: now also U9.5, U9.6 (NC); no longer U11.2, U11.9 (NC)
- net I2C3_SDA: now also U9.4, U9.7 (NC); no longer U9.2, U9.9 (NC)
- net I2C4_SCL: now also U11.2, U11.9 (NC); no longer U11.4, U11.7 (NC)
- net I2C4_SDA: now also U11.1, U11.10 (NC); no longer U9.4, U9.7 (NC)
- net I2C5_SDA: now also U11.4, U11.7 (NC); no longer U9.5, U9.6 (NC)
- net SOC_UART0_TX: now also U10.2, U10.9 (NC); no longer U12.1, U12.10 (NC)
- net SOC_UART1_RX: now also U10.4, U10.7 (NC); no longer U10.2, U10.9 (NC)
- net SOC_UART1_TX: now also U10.5, U10.6 (NC); no longer U12.2, U12.9 (NC)
- net SOC_UART2_RX: now also U12.1, U12.10 (NC); no longer U10.4, U10.7 (NC)
- net SOC_UART2_TX: now also U12.2, U12.9 (NC); no longer U12.4, U12.7 (NC)
- new net: U12.4, U12.7 (NC)
Changed lines of the file:
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@@
-	)
-	(label "SOC_UART1_TX"
-		(at 101.6 162.56 180)
-		(effects
-			(font
-				(size 1.27 1.27)
-			)
-			(justify right bottom)
-		)
 	)
 	(label "SOC_UART1_TX"
@@
 		)
 	)
-	(label "I2C3_SDA"
-		(at 38.1 73.66 180)
-		(effects
-			(font
-				(size 1.27 1.27)
-			)
-			(justify right bottom)
-		)
-	)
-	(label "SOC_UART1_RX"
-		(at 38.1 162.56 180)
-		(effects
-			(font
-				(size 1.27 1.27)
-			)
-			(justify right bottom)
+	(label "SOC_UART1_TX"
+		(at 63.5 162.56 0)
+		(effects
+			(font
+				(size 1.27 1.27)
+			)
+			(justify left bottom)
 		)
 	)
@@
 		)
 	)
-	(label "I2C4_SCL"
-		(at 127 68.58 0)
-		(effects
-			(font
-				(size 1.27 1.27)
-			)
-			(justify left bottom)
+	(label "SOC_UART2_RX"
+		(at 101.6 157.48 180)
+		(effects
+			(font
+				(size 1.27 1.27)
+			)
+			(justify right bottom)
 		)
 	)
@@
 		)
 	)
+	(label "SOC_UART2_TX"
+		(at 101.6 162.56 180)
+		(effects
+			(font
+				(size 1.27 1.27)
+			)
+			(justify right bottom)
+		)
+	)
 	(label "SOC_UART0_RX"
 		(at 44.45 127 0)
@@
 		)
 	)
-	(label "I2C5_SDA"
-		(at 63.5 73.66 0)
-		(effects
-			(font
-				(size 1.27 1.27)
-			)
-			(justify left bottom)
-		)
-	)
 	(label "SOC_UART0_TX"
 		(at 107.95 127 0)
@@
 		)
 	)
-	(label "SOC_UART0_TX"
-		(at 101.6 157.48 180)
-		(effects
-			(font
-				(size 1.27 1.27)
-			)
-			(justify right bottom)
+	(label "I2C5_SDA"
+		(at 127 68.58 0)
+		(effects
+			(font
+				(size 1.27 1.27)
+			)
+			(justify left bottom)
+		)
+	)
+	(label "SOC_UART1_RX"
+		(at 63.5 157.48 0)
+		(effects
+			(font
+				(size 1.27 1.27)
+			)
+			(justify left bottom)
 		)
 	)
@@
 		)
 	)
-	(label "SOC_UART2_TX"
-		(at 127 157.48 0)
-		(effects
-			(font
-				(size 1.27 1.27)
-			)
-			(justify left bottom)
-		)
-	)
 	(label "SOC_UART1_RX"
 		(at 44.45 129.54 0)
@@
 		)
 	)
-	(label "I2C4_SDA"
-		(at 63.5 68.58 0)
-		(effects
-			(font
-				(size 1.27 1.27)
-			)
-			(justify left bottom)
-		)
-	)
 	(label "I2C4_SCL"
 		(at 93.98 43.18 0)
@@
 		)
 	)
-	(label "I2C2_SCL"
-		(at 101.6 68.58 180)
-		(effects
-			(font
-				(size 1.27 1.27)
-			)
-			(justify right bottom)
-		)
-	)
-	(label "SOC_UART2_RX"
-		(at 63.5 157.48 0)
-		(effects
-			(font
-				(size 1.27 1.27)
-			)
-			(justify left bottom)
-		)
-	)
 	(label "I2C5_SCL"
 		(at 93.98 45.72 0)
@@
 	)
 	(label "I2C3_SCL"
-		(at 101.6 73.66 180)
-		(effects
-			(font
-				(size 1.27 1.27)
-			)
-			(justify right bottom)
+		(at 63.5 73.66 0)
+		(effects
+			(font
+				(size 1.27 1.27)
+			)
+			(justify left bottom)
+		)
+	)
+	(label "I2C2_SCL"
+		(at 38.1 73.66 180)
+		(effects
+			(font
+				(size 1.27 1.27)
+			)
+			(justify right bottom)
+		)
+	)
+	(label "SOC_UART0_TX"
+		(at 38.1 162.56 180)
+		(effects
+			(font
+				(size 1.27 1.27)
+			)
+			(justify right bottom)
+		)
+	)
+	(label "I2C4_SDA"
+		(at 101.6 68.58 180)
+		(effects
+			(font
+				(size 1.27 1.27)
+			)
+			(justify right bottom)
+		)
+	)
+	(label "I2C3_SDA"
+		(at 63.5 68.58 0)
+		(effects
+			(font
+				(size 1.27 1.27)
+			)
+			(justify left bottom)
 		)
 	)
@@
 		)
 	)
+	(label "I2C4_SCL"
+		(at 101.6 73.66 180)
+		(effects
+			(font
+				(size 1.27 1.27)
+			)
+			(justify right bottom)
+		)
+	)
